File: Hardware_v0/24V Regulator.sch (KiCad schematic (older format))
At the start: 0 parts

Commit message: Add +/-24V regulator design
Parts:
- added C? (x3): 10u, symbol Device:CP
- added C?: 0.1u, symbol Device:C
- added C?: 1u, symbol Device:CP
- added C?: 220p, symbol Device:C
- added C?: 0.2u, symbol Device:C
- added C?: 1u, symbol Device:C
- added D? (x2): NSR0530HT1G, symbol Device:D_Schottky
- added L? (x2): 15u, symbol Device:L
- added R?: 243K, symbol Device:R
- added R?: 4.12K, symbol Device:R
- added R?: 102K, symbol Device:R
- added R?: 3.16M, symbol Device:R
- added R?: 3.09M, symbol Device:R
- added R?: 107K, symbol Device:R
- added U?: ADP5070AREZ, Package_SO:ETSSOP-20-1EP_4.4x6.5mm_P0.65mm_EP3x4.2mm, symbol Regulator_Switching:ADP5070AREZ
Connections:
- new net: C?.1, U?.16 (VREG)
- new net: R?.1, U?.8 (COMP1)
- new net: C?.1, R?.2
- new net: C?.2, R?.1
- new net: R?.2, U?.12 (COMP2)
- new net: L?.1, U?.3 (INBK)
- new net: D?.2 (A), L?.2, U?.2 (SW1)
- new net: D?.1 (K), L?.1, U?.20 (SW2)
- new net: C?.1, R?.1, U?.14 (VREF)
- new net: R?.1, R?.2, U?.13 (FB2)
- new net: R?.1, R?.2, U?.7 (FB1)
- new net +24V: C?.1, D?.1 (K), R?.1
- new net -24V: C?.2, D?.2 (A), R?.2
- new net GND: C?.1, C?.1, C?.2, C?.2, C?.2, C?.2, C?.2, C?.2, L?.2, R?.2, U?.1 (PGND), U?.15 (AGND), U?.21 (AGND), U?.4 (SYNC/FREQ)
- new net Vin: C?.1, C?.1, U?.11 (EN2), U?.17 (PVIN1), U?.18 (PVINSYS), U?.19 (PVIN2), U?.9 (EN1)
- no-connect marks 0 -> 3
Other:
- note added: "+24V RAIL\n(500mA MAX)"
- note added: "-24V RAIL\n(500mA MAX)"
- note added: "Vin (3.3-12V)"
