File: Hardware_Device_Config_Demo/device-config-demo.sch (KiCad schematic (older format))
At the start: 91 parts, among them J1 0.1\" HDR, J2 0.1\" HDR, J3 0.1\" HDR, J4 0.1\" HDR, J5 0.1\" HDR, J6 0.1\" HDR, U1 ADA4522-4, U2 LTC6906, U3 MCP6002-xMS, U4 MCP4728A0

Commit message: Clean up device config demo board
Parts:
- removed U1: ADA4522-4, Package_SO:TSSOP-14_4.4x5mm_P0.65mm, symbol device-config-demo-rescue:ADA4522-4-io-master
- removed U2: LTC6906, Package_TO_SOT_SMD:TSOT-23-6, symbol device-config-demo-rescue:LTC6906-io-master
- added U1: ADA4522-4, Package_SO:TSSOP-14_4.4x5mm_P0.65mm, symbol io_master:ADA4522-4
- added U2: LTC6906, Package_TO_SOT_SMD:TSOT-23-6, symbol io_master:LTC6906
Connections:
- net +24V: now also U1.4 (V+)
- net +3V3: now also U2.6 (V+)
- net -24V: now also U1.11 (V-)
- net GND: now also U2.2 (GND), U2.3 (DIV)
- net VCO_OUT: now also U2.1 (OUT)
- net VH1: now also U1.1
- net VH2: now also U1.8
- net VL1: now also U1.7
- net VL2: now also U1.14
- net at R4.2, R5.1: now also U1.2 (-)
- net at R6.1, R7.2: now also U1.3 (+)
- net at R12.1, R14.2: now also U1.5 (+)
- net at R10.2, R11.1: now also U1.6 (-)
- net at R21.1, R22.2: now also U1.10 (+)
- net at R19.2, R20.1: now also U1.9 (-)
- net at R27.1, R28.2: now also U1.12 (+)
- net at R25.2, R26.1: now also U1.13 (-)
- net at R13.1: now also U2.4 (SET)
Changed lines of the file:
@@
 Text Notes 13200 2200 2    50   ~ 0
 VH1 = 1000/68 * (1.65V - Vdac)
-$Comp
-L device-config-demo-rescue:ADA4522-4-io-master U1
-U 5 1 5DC23D64
-P 13550 2700
-F 0 "U1" H 13508 2746 50  0001 L CNN
-F 1 "ADA4522-4" H 13508 2700 50  0001 L CNN
-F 2 "Package_SO:TSSOP-14_4.4x5mm_P0.65mm" H 13500 2800 50  0001 C CNN
-F 3 "https://www.analog.com/media/en/technical-documentation/data-sheets/ADA4522-1_4522-2_4522-4.pdf" H 13600 2900 50  0001 C CNN
-	5    13550 2700
-	1    0    0    -1
-$EndComp
-$Comp
-L device-config-demo-rescue:ADA4522-4-io-master U1
-U 1 1 5DC221CD
-P 13550 2700
-F 0 "U1" H 13550 2550 50  0000 L CNN
-F 1 "ADA4522-4" H 13550 2850 50  0000 L CNN
-F 2 "Package_SO:TSSOP-14_4.4x5mm_P0.65mm" H 13500 2800 50  0001 C CNN
-F 3 "https://www.analog.com/media/en/technical-documentation/data-sheets/ADA4522-1_4522-2_4522-4.pdf" H 13600 2900 50  0001 C CNN
-	1    13550 2700
-	1    0    0    1
-$EndComp
-$Comp
-L device-config-demo-rescue:ADA4522-4-io-master U1
-U 2 1 5DC2985B
-P 13550 4250
-F 0 "U1" H 13550 4100 50  0000 L CNN
-F 1 "ADA4522-4" H 13550 4400 50  0000 L CNN
-F 2 "Package_SO:TSSOP-14_4.4x5mm_P0.65mm" H 13500 4350 50  0001 C CNN
-F 3 "https://www.analog.com/media/en/technical-documentation/data-sheets/ADA4522-1_4522-2_4522-4.pdf" H 13600 4450 50  0001 C CNN
-	2    13550 4250
-	1    0    0    1
-$EndComp
-$Comp
-L device-config-demo-rescue:ADA4522-4-io-master U1
-U 4 1 5DC2AE59
-P 13550 7350
-F 0 "U1" H 13550 7200 50  0000 L CNN
-F 1 "ADA4522-4" H 13550 7500 50  0000 L CNN
-F 2 "Package_SO:TSSOP-14_4.4x5mm_P0.65mm" H 13500 7450 50  0001 C CNN
-F 3 "https://www.analog.com/media/en/technical-documentation/data-sheets/ADA4522-1_4522-2_4522-4.pdf" H 13600 7550 50  0001 C CNN
-	4    13550 7350
-	1    0    0    1
-$EndComp
-$Comp
-L device-config-demo-rescue:ADA4522-4-io-master U1
-U 3 1 5DC2A59A
-P 13550 5800
-F 0 "U1" H 13550 5650 50  0000 L CNN
-F 1 "ADA4522-4" H 13550 5950 50  0000 L CNN
-F 2 "Package_SO:TSSOP-14_4.4x5mm_P0.65mm" H 13500 5900 50  0001 C CNN
-F 3 "https://www.analog.com/media/en/technical-documentation/data-sheets/ADA4522-1_4522-2_4522-4.pdf" H 13600 6000 50  0001 C CNN
-	3    13550 5800
-	1    0    0    1
-$EndComp
 Wire Wire Line
 	12200 5700 12850 5700
@@
 Text Notes 750  3600 0    98   ~ 0
 VOLTAGE-CONTROLLED OSCILLATOR (VCO)
-$Comp
-L device-config-demo-rescue:LTC6906-io-master U2
-U 1 1 5DC77FBE
-P 5650 4500
-F 0 "U2" H 5400 4750 50  0000 C CNN
-F 1 "LTC6906" H 5850 4750 50  0000 C CNN
-F 2 "Package_TO_SOT_SMD:TSOT-23-6" H 5650 4500 98  0001 C CNN
-F 3 "" H 5650 4500 98  0001 C CNN
-	1    5650 4500
-	1    0    0    -1
-$EndComp
 $Comp
 L power:+3.3V #PWR0139
@@
 	-1   0    0    -1
 $EndComp
+$Comp
+L io_master:ADA4522-4 U1
+U 1 1 5DC5589D
+P 13550 2700
+F 0 "U1" H 13550 2550 50  0000 L CNN
+F 1 "ADA4522-4" H 13550 2850 50  0000 L CNN
+F 2 "Package_SO:TSSOP-14_4.4x5mm_P0.65mm" H 13500 2800 50  0001 C CNN
+F 3 "https://www.analog.com/media/en/technical-documentation/data-sheets/ADA4522-1_4522-2_4522-4.pdf" H 13600 2900 50  0001 C CNN
+	1    13550 2700
+	1    0    0    1
+$EndComp
+$Comp
+L io_master:ADA4522-4 U1
+U 5 1 5DC5BB84
+P 13550 2700
+F 0 "U1" H 13550 2850 50  0001 L CNN
+F 1 "ADA4522-4" H 13550 2550 50  0001 L CNN
+F 2 "Package_SO:TSSOP-14_4.4x5mm_P0.65mm" H 13500 2800 50  0001 C CNN
+F 3 "https://www.analog.com/media/en/technical-documentation/data-sheets/ADA4522-1_4522-2_4522-4.pdf" H 13600 2900 50  0001 C CNN
+	5    13550 2700
+	1    0    0    -1
+$EndComp
+$Comp
+L io_master:ADA4522-4 U1
+U 2 1 5DC6E8EE
+P 13550 4250
+F 0 "U1" H 13550 4100 50  0000 L CNN
+F 1 "ADA4522-4" H 13550 4400 50  0000 L CNN
+F 2 "Package_SO:TSSOP-14_4.4x5mm_P0.65mm" H 13500 4350 50  0001 C CNN
+F 3 "https://www.analog.com/media/en/technical-documentation/data-sheets/ADA4522-1_4522-2_4522-4.pdf" H 13600 4450 50  0001 C CNN
+	2    13550 4250
+	1    0    0    1
+$EndComp
+$Comp
+L io_master:ADA4522-4 U1
+U 3 1 5DC6EE6E
+P 13550 5800
+F 0 "U1" H 13550 5650 50  0000 L CNN
+F 1 "ADA4522-4" H 13550 5950 50  0000 L CNN
+F 2 "Package_SO:TSSOP-14_4.4x5mm_P0.65mm" H 13500 5900 50  0001 C CNN
+F 3 "https://www.analog.com/media/en/technical-documentation/data-sheets/ADA4522-1_4522-2_4522-4.pdf" H 13600 6000 50  0001 C CNN
+	3    13550 5800
+	1    0    0    1
+$EndComp
+$Comp
+L io_master:ADA4522-4 U1
+U 4 1 5DC6F478
+P 13550 7350
+F 0 "U1" H 13550 7200 50  0000 L CNN
+F 1 "ADA4522-4" H 13550 7500 50  0000 L CNN
+F 2 "Package_SO:TSSOP-14_4.4x5mm_P0.65mm" H 13500 7450 50  0001 C CNN
+F 3 "https://www.analog.com/media/en/technical-documentation/data-sheets/ADA4522-1_4522-2_4522-4.pdf" H 13600 7550 50  0001 C CNN
+	4    13550 7350
+	1    0    0    1
+$EndComp
+$Comp
+L io_master:LTC6906 U2
+U 1 1 5DC85267
+P 5650 4500
+F 0 "U2" H 5400 4750 50  0000 C CNN
+F 1 "LTC6906" H 5850 4750 50  0000 C CNN
+F 2 "Package_TO_SOT_SMD:TSOT-23-6" H 5650 4500 98  0001 C CNN
+F 3 "" H 5650 4500 98  0001 C CNN
+	1    5650 4500
+	1    0    0    -1
+$EndComp
 $EndSCHEMATC

Commit message: Update KiCAD symbol library
Parts:
- U1: symbol io_master:ADA4522-4 -> io-master:ADA4522-4
- U2: symbol io_master:LTC6906 -> io-master:LTC6906
Changed lines of the file:
@@
 $EndComp
 $Comp
-L io_master:ADA4522-4 U1
+L io-master:ADA4522-4 U1
 U 1 1 5DC5589D
 P 13550 2700
@@
 $EndComp
 $Comp
-L io_master:ADA4522-4 U1
+L io-master:ADA4522-4 U1
 U 5 1 5DC5BB84
 P 13550 2700
@@
 $EndComp
 $Comp
-L io_master:ADA4522-4 U1
+L io-master:ADA4522-4 U1
 U 2 1 5DC6E8EE
 P 13550 4250
@@
 $EndComp
 $Comp
-L io_master:ADA4522-4 U1
+L io-master:ADA4522-4 U1
 U 3 1 5DC6EE6E
 P 13550 5800
@@
 $EndComp
 $Comp
-L io_master:ADA4522-4 U1
+L io-master:ADA4522-4 U1
 U 4 1 5DC6F478
 P 13550 7350
@@
 $EndComp
 $Comp
-L io_master:LTC6906 U2
+L io-master:LTC6906 U2
 U 1 1 5DC85267
 P 5650 4500
