File: Hardware_Level_Shifter_Demo/level-shifter-demo.sch (KiCad schematic (older format))
At the start: 126 parts, among them J1 0.1\" HDR, J2 0.1\" HDR, J3 0.1\" HDR, J4 0.1\" HDR, J5 0.1\" HDR, Q1 2N7002, Q2 2N7002, Q3 2N7002, Q4 2N7002, Q5 2N7002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

Commit message: Update KiCAD symbol library
Parts:
- U2, U4: symbol io_master:ADA4522-4 -> io-master:ADA4522-4
- U3: symbol io_master:74AUP1T157 -> io-master:74AUP1T157
Changed lines of the file:
@@
 	13350 8700 13550 8700
 $Comp
-L io_master:74AUP1T157 U3
+L io-master:74AUP1T157 U3
 U 1 1 5DC61B79
 P 6100 2100
@@
 $EndComp
 $Comp
-L io_master:ADA4522-4 U2
+L io-master:ADA4522-4 U2
 U 1 1 5DC7DCD4
 P 7650 1950
@@
 $EndComp
 $Comp
-L io_master:ADA4522-4 U2
+L io-master:ADA4522-4 U2
 U 5 1 5DC7F804
 P 7850 1950
@@
 $EndComp
 $Comp
-L io_master:ADA4522-4 U2
+L io-master:ADA4522-4 U2
 U 2 1 5DC9D09A
 P 5950 4950
@@
 $EndComp
 $Comp
-L io_master:ADA4522-4 U4
+L io-master:ADA4522-4 U4
 U 1 1 5DC9E56E
 P 9150 4850
@@
 $EndComp
 $Comp
-L io_master:ADA4522-4 U4
+L io-master:ADA4522-4 U4
 U 2 1 5DC9ECAA
 P 7550 5450
@@
 $EndComp
 $Comp
-L io_master:ADA4522-4 U4
+L io-master:ADA4522-4 U4
 U 5 1 5DC9F28B
 P 9150 4850
@@
 $EndComp
 $Comp
-L io_master:ADA4522-4 U4
+L io-master:ADA4522-4 U4
 U 4 1 5DC9F69C
 P 5700 7250
@@
 $EndComp
 $Comp
-L io_master:ADA4522-4 U4
+L io-master:ADA4522-4 U4
 U 3 1 5DC9FEE6
 P 7550 6750
@@
 $EndComp
 $Comp
-L io_master:ADA4522-4 U2
+L io-master:ADA4522-4 U2
 U 4 1 5DCA045C
 P 5650 10050
@@
 $EndComp
 $Comp
-L io_master:ADA4522-4 U2
+L io-master:ADA4522-4 U2
 U 3 1 5DCD9D4B
 P 7550 9000
