File: KiCAD/Adjustable Regulator.sch (KiCad schematic (older format))
At the start: 17 parts, among them U4 LM2621

Commit message: Assign footprints, fix minor schematic issues
Parts:
- C40, C45: footprint Capacitor_SMD:C_1206_3216Metric -> Capacitor_SMD:C_1210_3225Metric
- C41, C46: footprint Capacitor_SMD:C_1206_3216Metric -> Capacitor_SMD:C_0805_2012Metric
- C42, C44: footprint Capacitor_SMD:C_1206_3216Metric -> Capacitor_SMD:C_0603_1608Metric
- C43: footprint (none) -> Capacitor_SMD:C_0603_1608Metric
- D13: footprint (none) -> Diode_SMD:D_SOD-323
- L1: footprint (none) -> io-master:L_Bourns_SRF0703
- R47, R48, R49: footprint (none) -> Resistor_SMD:R_0603_1608Metric
- TP108: value TestPoint -> SW; footprint (none) -> TestPoint:TestPoint_Pad_D1.0mm
- TP109: footprint (none) -> TestPoint:TestPoint_Pad_D1.0mm
- TP110: value TestPoint -> FB; footprint (none) -> TestPoint:TestPoint_Pad_D1.0mm
- TP111: value TestPoint -> Vout; footprint (none) -> TestPoint:TestPoint_Pad_D1.0mm
Changed lines of the file:
@@
 F 0 "L1" H 8150 5400 50  0000 C CNN
 F 1 "82u" H 8150 5300 50  0000 C CNN
-F 2 "" H 8150 5000 50  0001 C CNN
+F 2 "io-master:L_Bourns_SRF0703" H 8150 5000 50  0001 C CNN
 F 3 "~" H 8150 5000 50  0001 C CNN
 F 4 "SRF0703-820M" H 8150 5200 39  0000 C CNN "Device"
@@
 F 0 "C43" V 8498 4900 50  0000 C CNN
 F 1 "1u" V 8589 4900 50  0000 C CNN
-F 2 "" H 8788 4750 50  0001 C CNN
+F 2 "Capacitor_SMD:C_0603_1608Metric" H 8788 4750 50  0001 C CNN
 F 3 "~" H 8750 4900 50  0001 C CNN
 	1    8750 4900
@@
 F 0 "D13" H 9300 4684 50  0000 C CNN
 F 1 "NSR0530HT1G" H 9300 4775 39  0000 C CNN
-F 2 "" H 9300 4900 50  0001 C CNN
+F 2 "Diode_SMD:D_SOD-323" H 9300 4900 50  0001 C CNN
 F 3 "~" H 9300 4900 50  0001 C CNN
 	1    9300 4900
@@
 F 0 "R47" H 6100 5250 50  0000 R CNN
 F 1 "220K" H 6100 5150 50  0000 R CNN
-F 2 "" V 6130 5200 50  0001 C CNN
+F 2 "Resistor_SMD:R_0603_1608Metric" V 6130 5200 50  0001 C CNN
 F 3 "~" H 6200 5200 50  0001 C CNN
 	1    6200 5200
@@
 F 0 "C41" H 5615 5246 50  0000 L CNN
 F 1 "10u" H 5615 5155 50  0000 L CNN
-F 2 "Capacitor_SMD:C_1206_3216Metric" H 5538 5050 50  0001 C CNN
+F 2 "Capacitor_SMD:C_0805_2012Metric" H 5538 5050 50  0001 C CNN
 F 3 "~" H 5500 5200 50  0001 C CNN
 	1    5500 5200
@@
 F 0 "C40" H 5215 5246 50  0000 L CNN
 F 1 "C" H 5215 5155 50  0001 L CNN
-F 2 "Capacitor_SMD:C_1206_3216Metric" H 5138 5050 50  0001 C CNN
+F 2 "Capacitor_SMD:C_1210_3225Metric" H 5138 5050 50  0001 C CNN
 F 3 "~" H 5100 5200 50  0001 C CNN
 F 4 "DO NOT POP" V 4950 5200 39  0000 C CNN "Depop"
@@
 F 0 "C42" H 6765 5796 50  0000 L CNN
 F 1 "0.1u" H 6765 5705 50  0000 L CNN
-F 2 "Capacitor_SMD:C_1206_3216Metric" H 6688 5600 50  0001 C CNN
+F 2 "Capacitor_SMD:C_0603_1608Metric" H 6688 5600 50  0001 C CNN
 F 3 "~" H 6650 5750 50  0001 C CNN
 	1    6650 5750
@@
 F 0 "C46" H 11015 5246 50  0000 L CNN
 F 1 "10u" H 11015 5155 50  0000 L CNN
-F 2 "Capacitor_SMD:C_1206_3216Metric" H 10938 5050 50  0001 C CNN
+F 2 "Capacitor_SMD:C_0805_2012Metric" H 10938 5050 50  0001 C CNN
 F 3 "~" H 10900 5200 50  0001 C CNN
 	1    10900 5200
@@
 F 0 "C45" H 10615 5246 50  0000 L CNN
 F 1 "C" H 10615 5155 50  0001 L CNN
-F 2 "Capacitor_SMD:C_1206_3216Metric" H 10538 5050 50  0001 C CNN
+F 2 "Capacitor_SMD:C_1210_3225Metric" H 10538 5050 50  0001 C CNN
 F 3 "~" H 10500 5200 50  0001 C CNN
 F 4 "DO NOT POP" V 10350 5200 39  0000 C CNN "Depop"
@@
 F 0 "R48" H 9620 5396 50  0000 L CNN
 F 1 "110K" H 9620 5305 50  0000 L CNN
-F 2 "" V 9480 5350 50  0001 C CNN
+F 2 "Resistor_SMD:R_0603_1608Metric" V 9480 5350 50  0001 C CNN
 F 3 "~" H 9550 5350 50  0001 C CNN
 	1    9550 5350
@@
 F 0 "R49" H 9620 5796 50  0000 L CNN
 F 1 "10K" H 9620 5705 50  0000 L CNN
-F 2 "" V 9480 5750 50  0001 C CNN
+F 2 "Resistor_SMD:R_0603_1608Metric" V 9480 5750 50  0001 C CNN
 F 3 "~" H 9550 5750 50  0001 C CNN
 	1    9550 5750
@@
 F 0 "C44" H 10115 5396 50  0000 L CNN
 F 1 "33p" H 10115 5305 50  0000 L CNN
-F 2 "Capacitor_SMD:C_1206_3216Metric" H 10038 5200 50  0001 C CNN
+F 2 "Capacitor_SMD:C_0603_1608Metric" H 10038 5200 50  0001 C CNN
 F 3 "~" H 10000 5350 50  0001 C CNN
 	1    10000 5350
@@
 P 8500 4850
 F 0 "TP108" H 8500 5050 50  0000 C CNN
-F 1 "TestPoint" H 8558 4877 50  0001 L CNN
-F 2 "" H 8700 4850 50  0001 C CNN
+F 1 "SW" H 8558 4877 50  0001 L CNN
+F 2 "TestPoint:TestPoint_Pad_D1.0mm" H 8700 4850 50  0001 C CNN
 F 3 "~" H 8700 4850 50  0001 C CNN
 	1    8500 4850
@@
 F 0 "TP109" H 9000 5050 50  0000 C CNN
 F 1 "TestPoint" H 9058 4877 50  0001 L CNN
-F 2 "" H 9200 4850 50  0001 C CNN
+F 2 "TestPoint:TestPoint_Pad_D1.0mm" H 9200 4850 50  0001 C CNN
 F 3 "~" H 9200 4850 50  0001 C CNN
 	1    9000 4850
@@
 P 10900 4850
 F 0 "TP111" H 10900 5050 50  0000 C CNN
-F 1 "TestPoint" H 10958 4877 50  0001 L CNN
-F 2 "" H 11100 4850 50  0001 C CNN
+F 1 "Vout" H 10958 4877 50  0001 L CNN
+F 2 "TestPoint:TestPoint_Pad_D1.0mm" H 11100 4850 50  0001 C CNN
 F 3 "~" H 11100 4850 50  0001 C CNN
 	1    10900 4850
@@
 P 10000 5600
 F 0 "TP110" H 10000 5800 50  0000 C CNN
-F 1 "TestPoint" H 10058 5627 50  0001 L CNN
-F 2 "" H 10200 5600 50  0001 C CNN
+F 1 "FB" H 10058 5627 50  0001 L CNN
+F 2 "TestPoint:TestPoint_Pad_D1.0mm" H 10200 5600 50  0001 C CNN
 F 3 "~" H 10200 5600 50  0001 C CNN
 	1    10000 5600
