File: KiCAD/Circuit Protection - IO 2.sch (KiCad schematic (older format))
At the start: 28 parts, among them Q25 DMN63D8LDW, Q26 MMBT3906, U37 NCV20074

Commit message: Assign footprints, fix minor schematic issues
Parts:
- C117, C118: footprint (none) -> Capacitor_SMD:C_0603_1608Metric
- D33, D34, D38, D39: footprint (none) -> Diode_SMD:D_SOD-323
- D35: footprint (none) -> LED_SMD:LED_0603_1608Metric
- Q26: footprint Package_TO_SOT_SMD:SOT-23 -> Package_TO_SOT_SMD:SOT-323_SC-70
- R247, R248, R249, R250, R251, R252, R253, R254, R255, R256, R257, R258, R259, R260, R261: footprint (none) -> Resistor_SMD:R_0603_1608Metric
- TP171, TP172, TP173: footprint (none) -> TestPoint:TestPoint_Pad_D1.0mm
Changed lines of the file:
@@
 F 0 "D33" V 9996 5171 50  0000 R CNN
 F 1 "1N4148" V 9905 5171 50  0000 R CNN
-F 2 "" H 9950 5250 50  0001 C CNN
+F 2 "Diode_SMD:D_SOD-323" H 9950 5250 50  0001 C CNN
 F 3 "~" H 9950 5250 50  0001 C CNN
 	1    9950 5250
@@
 F 0 "R259" H 12570 4596 50  0000 L CNN
 F 1 "100K" H 12570 4505 50  0000 L CNN
-F 2 "" V 12430 4550 50  0001 C CNN
+F 2 "Resistor_SMD:R_0603_1608Metric" V 12430 4550 50  0001 C CNN
 F 3 "~" H 12500 4550 50  0001 C CNN
 	1    12500 4550
@@
 F 0 "R250" H 7750 5750 50  0000 L CNN
 F 1 "100K" H 7750 5650 50  0000 L CNN
-F 2 "" V 7630 5700 50  0001 C CNN
+F 2 "Resistor_SMD:R_0603_1608Metric" V 7630 5700 50  0001 C CNN
 F 3 "~" H 7700 5700 50  0001 C CNN
 	1    7700 5700
@@
 F 0 "R249" V 7400 5450 50  0000 C CNN
 F 1 "10K" V 7500 5450 50  0000 C CNN
-F 2 "" V 7430 5450 50  0001 C CNN
+F 2 "Resistor_SMD:R_0603_1608Metric" V 7430 5450 50  0001 C CNN
 F 3 "~" H 7500 5450 50  0001 C CNN
 	1    7500 5450
@@
 F 0 "R251" V 7950 4850 50  0000 C CNN
 F 1 "100K" V 8050 4850 50  0000 C CNN
-F 2 "" V 7980 4850 50  0001 C CNN
+F 2 "Resistor_SMD:R_0603_1608Metric" V 7980 4850 50  0001 C CNN
 F 3 "~" H 8050 4850 50  0001 C CNN
 	1    8050 4850
@@
 F 0 "R248" V 7400 5250 50  0000 C CNN
 F 1 "10K" V 7500 5250 50  0000 C CNN
-F 2 "" V 7430 5250 50  0001 C CNN
+F 2 "Resistor_SMD:R_0603_1608Metric" V 7430 5250 50  0001 C CNN
 F 3 "~" H 7500 5250 50  0001 C CNN
 	1    7500 5250
@@
 F 0 "R252" V 8650 5350 50  0000 C CNN
 F 1 "100K" V 8750 5350 50  0000 C CNN
-F 2 "" V 8680 5350 50  0001 C CNN
+F 2 "Resistor_SMD:R_0603_1608Metric" V 8680 5350 50  0001 C CNN
 F 3 "~" H 8750 5350 50  0001 C CNN
 	1    8750 5350
@@
 F 0 "R253" V 9350 5050 50  0000 C CNN
 F 1 "100K" V 9450 5050 50  0000 C CNN
-F 2 "" V 9380 5050 50  0001 C CNN
+F 2 "Resistor_SMD:R_0603_1608Metric" V 9380 5050 50  0001 C CNN
 F 3 "~" H 9450 5050 50  0001 C CNN
 	1    9450 5050
@@
 F 0 "R254" V 9350 5900 50  0000 C CNN
 F 1 "100K" V 9450 5900 50  0000 C CNN
-F 2 "" V 9380 5900 50  0001 C CNN
+F 2 "Resistor_SMD:R_0603_1608Metric" V 9380 5900 50  0001 C CNN
 F 3 "~" H 9450 5900 50  0001 C CNN
 	1    9450 5900
@@
 F 0 "R255" V 10100 5050 50  0000 C CNN
 F 1 "100K" V 10200 5050 50  0000 C CNN
-F 2 "" V 10130 5050 50  0001 C CNN
+F 2 "Resistor_SMD:R_0603_1608Metric" V 10130 5050 50  0001 C CNN
 F 3 "~" H 10200 5050 50  0001 C CNN
 	1    10200 5050
@@
 F 0 "R256" V 10650 5050 50  0000 C CNN
 F 1 "100K" V 10750 5050 50  0000 C CNN
-F 2 "" V 10680 5050 50  0001 C CNN
+F 2 "Resistor_SMD:R_0603_1608Metric" V 10680 5050 50  0001 C CNN
 F 3 "~" H 10750 5050 50  0001 C CNN
 	1    10750 5050
@@
 F 0 "R257" H 11400 6350 50  0000 L CNN
 F 1 "100K" H 11400 6250 50  0000 L CNN
-F 2 "" V 11280 6300 50  0001 C CNN
+F 2 "Resistor_SMD:R_0603_1608Metric" V 11280 6300 50  0001 C CNN
 F 3 "~" H 11350 6300 50  0001 C CNN
 	1    11350 6300
@@
 F 0 "R258" H 11400 6750 50  0000 L CNN
 F 1 "6.8K" H 11400 6650 50  0000 L CNN
-F 2 "" V 11280 6700 50  0001 C CNN
+F 2 "Resistor_SMD:R_0603_1608Metric" V 11280 6700 50  0001 C CNN
 F 3 "~" H 11350 6700 50  0001 C CNN
 	1    11350 6700
@@
 F 0 "D34" V 9996 5571 50  0000 R CNN
 F 1 "1N4148" V 9905 5571 50  0000 R CNN
-F 2 "" H 9950 5650 50  0001 C CNN
+F 2 "Diode_SMD:D_SOD-323" H 9950 5650 50  0001 C CNN
 F 3 "~" H 9950 5650 50  0001 C CNN
 	1    9950 5650
@@
 F 0 "D35" V 13639 5832 50  0000 R CNN
 F 1 "RED" V 13548 5832 50  0000 R CNN
-F 2 "" H 13600 5950 50  0001 C CNN
+F 2 "LED_SMD:LED_0603_1608Metric" H 13600 5950 50  0001 C CNN
 F 3 "~" H 13600 5950 50  0001 C CNN
 	1    13600 5950
@@
 F 0 "R261" H 13670 6346 50  0000 L CNN
 F 1 "10K" H 13670 6255 50  0000 L CNN
-F 2 "" V 13530 6300 50  0001 C CNN
+F 2 "Resistor_SMD:R_0603_1608Metric" V 13530 6300 50  0001 C CNN
 F 3 "~" H 13600 6300 50  0001 C CNN
 	1    13600 6300
@@
 F 0 "R260" V 13000 5550 50  0000 C CNN
 F 1 "10K" V 13100 5550 50  0000 C CNN
-F 2 "" V 13030 5550 50  0001 C CNN
+F 2 "Resistor_SMD:R_0603_1608Metric" V 13030 5550 50  0001 C CNN
 F 3 "~" H 13100 5550 50  0001 C CNN
 	1    13100 5550
@@
 F 0 "Q26" H 13500 5400 50  0000 R CNN
 F 1 "MMBT3906" H 13500 5700 50  0000 R CNN
-F 2 "Package_TO_SOT_SMD:SOT-23" H 13700 5475 50  0001 L CIN
+F 2 "Package_TO_SOT_SMD:SOT-323_SC-70" H 13700 5475 50  0001 L CIN
 F 3 "https://www.fairchildsemi.com/datasheets/2N/2N3906.pdf" H 13500 5550 50  0001 L CNN
 	1    13500 5550
@@
 F 0 "R247" V 7000 4350 50  0000 C CNN
 F 1 "2" V 7100 4350 50  0000 C CNN
-F 2 "" V 7030 4350 50  0001 C CNN
+F 2 "Resistor_SMD:R_0603_1608Metric" V 7030 4350 50  0001 C CNN
 F 3 "~" H 7100 4350 50  0001 C CNN
 	1    7100 4350
@@
 F 0 "TP171" V 8450 5038 50  0000 L CNN
 F 1 "TestPoint" V 8495 5038 50  0001 L CNN
-F 2 "" H 8650 4850 50  0001 C CNN
+F 2 "TestPoint:TestPoint_Pad_D1.0mm" H 8650 4850 50  0001 C CNN
 F 3 "~" H 8650 4850 50  0001 C CNN
 	1    8450 4850
@@
 F 0 "TP172" V 11250 5238 50  0000 L CNN
 F 1 "TestPoint" V 11295 5238 50  0001 L CNN
-F 2 "" H 11450 5050 50  0001 C CNN
+F 2 "TestPoint:TestPoint_Pad_D1.0mm" H 11450 5050 50  0001 C CNN
 F 3 "~" H 11450 5050 50  0001 C CNN
 	1    11250 5050
@@
 F 0 "TP173" H 12500 5850 50  0000 C TNN
 F 1 "TestPoint" V 12545 5788 50  0001 L CNN
-F 2 "" H 12700 5600 50  0001 C CNN
+F 2 "TestPoint:TestPoint_Pad_D1.0mm" H 12700 5600 50  0001 C CNN
 F 3 "~" H 12700 5600 50  0001 C CNN
 	1    12500 5600
@@
 F 0 "D39" V 3950 4850 50  0000 R CNN
 F 1 "MM3Z15VST1G" V 4050 4850 50  0000 R CNN
-F 2 "" H 4000 4950 50  0001 C CNN
+F 2 "Diode_SMD:D_SOD-323" H 4000 4950 50  0001 C CNN
 F 3 "~" H 4000 4950 50  0001 C CNN
 	1    4000 4950
@@
 F 0 "D38" V 4050 4500 50  0000 R CNN
 F 1 "MM3Z15VST1G" V 3950 4500 50  0000 R CNN
-F 2 "" H 4000 4600 50  0001 C CNN
+F 2 "Diode_SMD:D_SOD-323" H 4000 4600 50  0001 C CNN
 F 3 "~" H 4000 4600 50  0001 C CNN
 	1    4000 4600
@@
 F 0 "C117" H 8565 3096 50  0000 L CNN
 F 1 "0.1u" H 8565 3005 50  0000 L CNN
-F 2 "" H 8488 2900 50  0001 C CNN
+F 2 "Capacitor_SMD:C_0603_1608Metric" H 8488 2900 50  0001 C CNN
 F 3 "~" H 8450 3050 50  0001 C CNN
 	1    8450 3050
@@
 F 0 "C118" H 8565 3496 50  0000 L CNN
 F 1 "0.1u" H 8565 3405 50  0000 L CNN
-F 2 "" H 8488 3300 50  0001 C CNN
+F 2 "Capacitor_SMD:C_0603_1608Metric" H 8488 3300 50  0001 C CNN
 F 3 "~" H 8450 3450 50  0001 C CNN
 	1    8450 3450
