File: KiCAD/io-master.sch (KiCad schematic (older format))
At the start: 49 parts, among them J1 Jack-DC, J2 USB_B_Micro, J3 0.1\" HDR, Q1 Q_NPN_BCE, Q2 Q_NPN_BCE, U1 AZ1117-3.3

Commit message: Add power changeover circuit, fix minor issues
Parts:
- added Q27: DMP3099L, symbol Device:Q_PMOS_GSD
- added R262: 100K, symbol Device:R
- D1, D2: value SS14FL -> B130L
- J1: value Jack-DC -> PJ-037A
- J2: value USB_B_Micro -> 10118193
- TP4: value KEYSTONE 5011 -> GND; Device (none) -> KEYSTONE 5011
Connections:
- net GND: now also R262.2
- net Microcontroller/USB_VBUS: now also Q27.2 (S); no longer D2.2 (A)
- net at D1.2 (A), J1.1, TP17.1: now also Q27.1 (G), R262.1
- new net: D2.2 (A), Q27.3 (D)
Other:
- note added: "INPUT: 4.6-15V"
- note added: "USB 2.0 INPUT\n(5V, 500mA)"
- note removed: "USB 2.0\nTO COMPUTER\n(5V, 500mA)"
- moved on the sheet: C2, D2, TP17, TP18
Changed lines of the file:
@@
 Sheet 1 10
 Title "I/O MASTER v1"
-Date "2020-02-03"
+Date "2020-02-04"
 Rev "A"
 Comp "THE UNIVERSITY OF AKRON"
@@
 $EndSheet
 $Comp
-L Connector:Jack-DC J1
-U 1 1 5DA50F70
-P 2200 3000
-F 0 "J1" H 2200 3300 50  0000 C CNN
-F 1 "Jack-DC" H 2200 3200 50  0000 C CNN
-F 2 "" H 2250 2960 50  0001 C CNN
-F 3 "~" H 2250 2960 50  0001 C CNN
-	1    2200 3000
-	1    0    0    -1
-$EndComp
-$Comp
 L power:GND #PWR04
 U 1 1 5DA51E3F
-P 2550 3150
-F 0 "#PWR04" H 2550 2900 50  0001 C CNN
-F 1 "GND" H 2555 2977 50  0000 C CNN
-F 2 "" H 2550 3150 50  0001 C CNN
-F 3 "" H 2550 3150 50  0001 C CNN
-	1    2550 3150
-	1    0    0    -1
-$EndComp
-Wire Wire Line
-	2500 3100 2550 3100
-Wire Wire Line
-	2550 3100 2550 3150
-Text Notes 1900 4150 2    79   ~ 0
-USB 2.0\nTO COMPUTER\n(5V, 500mA)
+P 2700 3150
+F 0 "#PWR04" H 2700 2900 50  0001 C CNN
+F 1 "GND" H 2705 2977 50  0000 C CNN
+F 2 "" H 2700 3150 50  0001 C CNN
+F 3 "" H 2700 3150 50  0001 C CNN
+	1    2700 3150
+	1    0    0    -1
+$EndComp
+Wire Wire Line
+	2500 3100 2700 3100
+Wire Wire Line
+	2700 3100 2700 3150
+Text Notes 1900 4100 2    79   ~ 0
+USB 2.0 INPUT\n(5V, 500mA)
 Text Notes 1900 3100 2    79   ~ 0
 OPTIONAL DC INPUT\n(12V, 500mA)
@@
 	2500 2900 2550 2900
 Wire Wire Line
-	2550 2900 2550 2450
-Wire Wire Line
-	2850 3800 2850 2450
-Wire Wire Line
-	2850 1950 2850 1850
-Wire Wire Line
-	2850 1850 2550 1850
+	2550 2900 2550 2500
+Wire Wire Line
+	3050 3800 3050 3450
+Wire Wire Line
+	3050 1950 3050 1850
+Wire Wire Line
+	3050 1850 2550 1850
 Wire Wire Line
 	2550 1850 2550 1950
@@
 L power:GND #PWR06
 U 1 1 5FD56646
-P 2850 4500
-F 0 "#PWR06" H 2850 4250 50  0001 C CNN
-F 1 "GND" H 2855 4327 50  0000 C CNN
-F 2 "" H 2850 4500 50  0001 C CNN
-F 3 "" H 2850 4500 50  0001 C CNN
-	1    2850 4500
+P 3050 4500
+F 0 "#PWR06" H 3050 4250 50  0001 C CNN
+F 1 "GND" H 3055 4327 50  0000 C CNN
+F 2 "" H 3050 4500 50  0001 C CNN
+F 3 "" H 3050 4500 50  0001 C CNN
+	1    3050 4500
 	1    0    0    -1
 $EndComp
@@
 L Device:C C2
 U 1 1 5FD56659
-P 2850 4300
-F 0 "C2" H 2965 4346 50  0000 L CNN
-F 1 "1uF" H 2965 4255 50  0000 L CNN
-F 2 "" H 2888 4150 50  0001 C CNN
-F 3 "~" H 2850 4300 50  0001 C CNN
-	1    2850 4300
+P 3050 4300
+F 0 "C2" H 3165 4346 50  0000 L CNN
+F 1 "1uF" H 3165 4255 50  0000 L CNN
+F 2 "" H 3088 4150 50  0001 C CNN
+F 3 "~" H 3050 4300 50  0001 C CNN
+	1    3050 4300
 	1    0    0    -1
 $EndComp
@@
 U 1 1 5FD5665F
 P 2200 4000
-F 0 "J2" H 2257 4467 50  0000 C CNN
-F 1 "USB_B_Micro" H 2257 4376 50  0000 C CNN
+F 0 "J2" H 2200 4450 50  0000 C CNN
+F 1 "10118193" H 2200 4350 50  0000 C CNN
 F 2 "" H 2350 3950 50  0001 C CNN
 F 3 "~" H 2350 3950 50  0001 C CNN
@@
 $EndComp
 Wire Wire Line
-	2850 4450 2850 4500
+	3050 4450 3050 4500
 NoConn ~ 2500 4200
 $Comp
@@
 $EndComp
 Wire Wire Line
-	2500 3800 2850 3800
-Connection ~ 2850 3800
+	2500 3800 3050 3800
+Connection ~ 3050 3800
 Wire Wire Line
 	2500 4000 4000 4000
@@
 	2500 4100 4000 4100
 Wire Wire Line
-	2850 3800 2850 4150
-Wire Wire Line
-	2850 3800 4000 3800
+	3050 3800 3050 4150
+Wire Wire Line
+	3050 3800 4000 3800
 $Comp
 L Device:D_Schottky D2
 U 1 1 609C9840
-P 2850 2100
-F 0 "D2" V 2804 2179 50  0000 L CNN
-F 1 "SS14FL" V 2895 2179 50  0000 L CNN
-F 2 "" H 2850 2100 50  0001 C CNN
-F 3 "~" H 2850 2100 50  0001 C CNN
-	1    2850 2100
+P 3050 2100
+F 0 "D2" V 3004 2179 50  0000 L CNN
+F 1 "B130L" V 3095 2179 50  0000 L CNN
+F 2 "" H 3050 2100 50  0001 C CNN
+F 3 "~" H 3050 2100 50  0001 C CNN
+	1    3050 2100
 	0    1    1    0
 $EndComp
@@
 P 2550 2100
 F 0 "D1" V 2500 2000 50  0000 R CNN
-F 1 "SS14FL" V 2600 2000 50  0000 R CNN
+F 1 "B130L" V 2600 2000 50  0000 R CNN
 F 2 "" H 2550 2100 50  0001 C CNN
 F 3 "~" H 2550 2100 50  0001 C CNN
@@
 U 1 1 5E450097
 P 1250 1700
-F 0 "TP4" H 1308 1810 50  0000 L CNN
-F 1 "KEYSTONE 5011" H 1308 1727 39  0000 L CNN
+F 0 "TP4" H 1250 2000 50  0000 C CNN
+F 1 "GND" H 1308 1727 50  0001 L CNN
 F 2 "" H 1450 1700 50  0001 C CNN
 F 3 "~" H 1450 1700 50  0001 C CNN
+F 4 "KEYSTONE 5011" H 1250 1950 39  0000 C TNN "Device"
 	1    1250 1700
 	1    0    0    -1
@@
 L Connector:TestPoint TP17
 U 1 1 5F5A4C4A
-P 2500 2450
-F 0 "TP17" V 2500 2650 50  0000 L CNN
-F 1 "TestPoint" V 2604 2522 50  0001 C CNN
-F 2 "" H 2700 2450 50  0001 C CNN
-F 3 "~" H 2700 2450 50  0001 C CNN
-	1    2500 2450
+P 2500 2500
+F 0 "TP17" V 2500 2700 50  0000 L CNN
+F 1 "TestPoint" V 2604 2572 50  0001 C CNN
+F 2 "" H 2700 2500 50  0001 C CNN
+F 3 "~" H 2700 2500 50  0001 C CNN
+	1    2500 2500
 	0    -1   -1   0
 $EndComp
@@
 L Connector:TestPoint TP18
 U 1 1 5F5A526A
-P 2900 2450
-F 0 "TP18" V 2900 2650 50  0000 L CNN
-F 1 "TestPoint" V 3004 2522 50  0001 C CNN
-F 2 "" H 3100 2450 50  0001 C CNN
-F 3 "~" H 3100 2450 50  0001 C CNN
-	1    2900 2450
+P 3100 3450
+F 0 "TP18" V 3100 3650 50  0000 L CNN
+F 1 "TestPoint" V 3204 3522 50  0001 C CNN
+F 2 "" H 3300 3450 50  0001 C CNN
+F 3 "~" H 3300 3450 50  0001 C CNN
+	1    3100 3450
 	0    1    -1   0
 $EndComp
 Wire Wire Line
-	2850 2450 2900 2450
-Connection ~ 2850 2450
-Wire Wire Line
-	2850 2450 2850 2250
-Wire Wire Line
-	2500 2450 2550 2450
-Connection ~ 2550 2450
-Wire Wire Line
-	2550 2450 2550 2250
+	3050 2300 3050 2250
 $Comp
 L io-master:CHASSIS #PWR0149
@@
 Wire Wire Line
 	16100 9050 16150 9050
+$Comp
+L Device:Q_PMOS_GSD Q27
+U 1 1 5E527EDC
+P 2950 2500
+F 0 "Q27" H 3154 2546 50  0000 L CNN
+F 1 "DMP3099L" H 3154 2455 50  0000 L CNN
+F 2 "" H 3150 2600 50  0001 C CNN
+F 3 "~" H 2950 2500 50  0001 C CNN
+	1    2950 2500
+	1    0    0    -1
+$EndComp
+$Comp
+L Device:R R262
+U 1 1 5E568682
+P 2700 2800
+F 0 "R262" H 2770 2846 50  0000 L CNN
+F 1 "100K" H 2770 2755 50  0000 L CNN
+F 2 "" V 2630 2800 50  0001 C CNN
+F 3 "~" H 2700 2800 50  0001 C CNN
+	1    2700 2800
+	1    0    0    -1
+$EndComp
+Wire Wire Line
+	2700 3100 2700 2950
+Connection ~ 2700 3100
+Wire Wire Line
+	2750 2500 2700 2500
+Wire Wire Line
+	2700 2500 2700 2650
+Wire Wire Line
+	2700 2500 2550 2500
+Connection ~ 2700 2500
+Connection ~ 2550 2500
+Wire Wire Line
+	2550 2250 2550 2500
+Wire Wire Line
+	2500 2500 2550 2500
+Wire Wire Line
+	3100 3450 3050 3450
+Connection ~ 3050 3450
+Wire Wire Line
+	3050 3450 3050 2700
+$Comp
+L Connector:Jack-DC J1
+U 1 1 5DA50F70
+P 2200 3000
+F 0 "J1" H 2200 3300 50  0000 C CNN
+F 1 "PJ-037A" H 2200 3200 50  0000 C CNN
+F 2 "" H 2250 2960 50  0001 C CNN
+F 3 "~" H 2250 2960 50  0001 C CNN
+	1    2200 3000
+	1    0    0    -1
+$EndComp
+Text Notes 3900 1650 0    50   ~ 0
+INPUT: 4.6-15V
 $EndSCHEMATC

Commit message: Change barrel jack to cheaper part, add footprint
Parts:
- removed J1: PJ-037A, symbol Connector:Jack-DC
- added J1: 54-00166, io-master:BarrelJack_Tensility_54-00166_Horizontal, symbol Connector:Barrel_Jack_Switch
Connections:
- net GND: now also J1.2, J1.3
- net at D1.2 (A), Q27.1 (G), R262.1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: now also J1.1
Changed lines of the file:
@@
 Sheet 1 10
 Title "I/O MASTER v1"
-Date "2020-02-04"
+Date "2020-02-05"
 Rev "A"
 Comp "THE UNIVERSITY OF AKRON"
@@
 $EndComp
 Wire Wire Line
-	2500 3100 2700 3100
+	2500 3100 2550 3100
 Wire Wire Line
 	2700 3100 2700 3150
@@
 Wire Wire Line
 	3050 3450 3050 2700
-$Comp
-L Connector:Jack-DC J1
-U 1 1 5DA50F70
+Text Notes 3900 1650 0    50   ~ 0
+INPUT: 4.6-15V
+$Comp
+L Connector:Barrel_Jack_Switch J1
+U 1 1 5E3C0817
 P 2200 3000
 F 0 "J1" H 2200 3300 50  0000 C CNN
-F 1 "PJ-037A" H 2200 3200 50  0000 C CNN
-F 2 "" H 2250 2960 50  0001 C CNN
-F 3 "~" H 2250 2960 50  0001 C CNN
+F 1 "54-00166" H 2200 3200 50  0000 C CNN
+F 2 "io-master:BarrelJack_Tensility_54-00166_Horizontal" H 2250 2960 50  0001 C CNN
+F 3 "https://tensility.s3.amazonaws.com/uploads/pdffiles/54-00166.pdf?X-Amz-Expires=600&X-Amz-Date=20200205T184808Z&X-Amz-Algorithm=AWS4-HMAC-SHA256&X-Amz-Credential=AKIAIS2S4WRDQDSWDRZQ%2F20200205%2Fus-west-2%2Fs3%2Faws4_request&X-Amz-SignedHeaders=host&X-Amz-Signature=cee2821c2b89355b72751d43bd97aff6d341b62e1b5ea29893536d159c2204cc" H 2250 2960 50  0001 C CNN
 	1    2200 3000
 	1    0    0    -1
 $EndComp
-Text Notes 3900 1650 0    50   ~ 0
-INPUT: 4.6-15V
+Wire Wire Line
+	2500 3000 2550 3000
+Wire Wire Line
+	2550 3000 2550 3100
+Connection ~ 2550 3100
+Wire Wire Line
+	2550 3100 2700 3100
 $EndSCHEMATC

Commit message: Assign footprints, fix minor schematic issues
Parts:
- C1, C2, C3, C6: footprint (none) -> Capacitor_SMD:C_0603_1608Metric
- C4: footprint (none) -> Capacitor_SMD:C_0805_2012Metric
- C5: footprint (none) -> Capacitor_SMD:C_1210_3225Metric
- D1, D2: footprint (none) -> Diode_SMD:D_SMA
- D3, D4, D5, D6: footprint (none) -> LED_SMD:LED_0603_1608Metric
- H1, H2, H3, H4: footprint (none) -> MountingHole:MountingHole_3.2mm_M3_Pad
- J2: footprint (none) -> io-master:USB_Micro-B_Amphenol_10118193-0001LF_Horizontal
- J3: footprint (none) -> Connector_PinSocket_2.54mm:PinSocket_2x05_P2.54mm_Vertical
- Q1, Q2: footprint (none) -> Package_TO_SOT_SMD:SOT-323_SC-70
- Q27: footprint (none) -> Package_TO_SOT_SMD:SOT-23
- R1, R2, R262, R3, R4, R5, R6, R7, R8: footprint (none) -> Resistor_SMD:R_0603_1608Metric
- TP1, TP10, TP11, TP12, TP13, TP14, TP15, TP17, TP2, TP3, TP5, TP6, TP7, TP8, TP9: footprint (none) -> TestPoint:TestPoint_Pad_D1.0mm
- TP16: value TestPoint -> VIN; footprint (none) -> TestPoint:TestPoint_Pad_D1.0mm
- TP18: value TestPoint -> VBUS; footprint (none) -> TestPoint:TestPoint_Pad_D1.0mm
- TP19: value TestPoint -> 3.3V; footprint (none) -> TestPoint:TestPoint_Pad_D1.0mm
- TP4: footprint (none) -> TestPoint:TestPoint_Keystone_5010-5014_Multipurpose
- U1: footprint (none) -> Package_TO_SOT_SMD:SOT-223-3_TabPin2

Commit message: Add PTC fuses on Vin and Vout
Parts:
- added F1: 0.5A, Fuse:Fuse_1206_3216Metric, symbol Device:Polyfuse
- added F2: 0.1A, Fuse:Fuse_1206_3216Metric, symbol Device:Polyfuse
Connections:
- net Vin: now also F1.1; no longer D1.1 (K), D2.1 (K)
- net Vout: now also F2.2
- new net: D1.1 (K), D2.1 (K), F1.2
- new net Adjustable Regulator/Vout: F2.1
Changed lines of the file:
@@
 Sheet 1 10
 Title "I/O MASTER v1"
-Date "2020-02-05"
+Date "2020-02-07"
 Rev "A"
 Comp "THE UNIVERSITY OF AKRON"
@@
 	6700 1250 3850 1250
 Wire Wire Line
-	2550 1250 2550 1850
+	2550 1250 2550 1400
 Wire Wire Line
 	3850 1800 3850 1250
@@
 	13850 6300 13950 6300
 Wire Wire Line
-	13850 4850 13850 6300
+	13850 4850 13850 5100
 Wire Wire Line
 	15150 4000 15350 4000
@@
 Wire Wire Line
 	2550 3100 2700 3100
+Wire Wire Line
+	13850 5400 13850 6300
+Wire Wire Line
+	2550 1700 2550 1850
+$Comp
+L Device:Polyfuse F1
+U 1 1 5E3F0B3D
+P 2550 1550
+F 0 "F1" H 2638 1596 50  0000 L CNN
+F 1 "0.5A" H 2638 1505 50  0000 L CNN
+F 2 "Fuse:Fuse_1206_3216Metric" H 2600 1350 50  0001 L CNN
+F 3 "~" H 2550 1550 50  0001 C CNN
+	1    2550 1550
+	1    0    0    -1
+$EndComp
+$Comp
+L Device:Polyfuse F2
+U 1 1 5E3F2C3B
+P 13850 5250
+F 0 "F2" H 13938 5296 50  0000 L CNN
+F 1 "0.1A" H 13938 5205 50  0000 L CNN
+F 2 "Fuse:Fuse_1206_3216Metric" H 13900 5050 50  0001 L CNN
+F 3 "~" H 13850 5250 50  0001 C CNN
+	1    13850 5250
+	1    0    0    -1
+$EndComp
 $EndSCHEMATC

Commit message: Add C18 and C21 0.1u decoupling caps, fix minor issues
Parts:
- J3: footprint Connector_PinSocket_2.54mm:PinSocket_2x05_P2.54mm_Vertical -> io-master:PinSocket_2x05_P2.54mm_Vertical_AltNumbering
- TP17: value TestPoint -> DCIN
Connections:
- net Adjustable Regulator/Vout is gone; now on net Vout: F2.1
- net Vout: no longer F2.2, J3.5 (Pin_5)
- new net: F2.2, J3.5 (Pin_5)
Other:
- moved on the sheet: F2
Changed lines of the file:
@@
 Sheet 1 10
 Title "I/O MASTER v1"
-Date "2020-02-07"
+Date "2020-02-10"
 Rev "A"
 Comp "THE UNIVERSITY OF AKRON"
@@
 	6700 2000 6700 1250
 Wire Wire Line
-	6700 1250 3850 1250
-Wire Wire Line
 	2550 1250 2550 1400
 Wire Wire Line
-	3850 1800 3850 1250
-Connection ~ 3850 1250
-Wire Wire Line
-	3850 1250 2550 1250
-Wire Wire Line
 	8700 2050 8700 3100
 Wire Wire Line
 	8800 1950 8800 3000
 Wire Wire Line
-	15350 4000 15350 4850
-Wire Wire Line
-	15350 4850 13850 4850
+	15350 4000 15350 5050
+Wire Wire Line
+	15350 5050 13850 5050
 Wire Wire Line
 	6700 1250 13300 1250
@@
 Connection ~ 3850 2200
 Connection ~ 5650 1800
-Connection ~ 3850 1800
-Text Label 3900 1800 0    50   ~ 0
-Vin
 Wire Notes Line
 	3650 1500 3650 2500
@@
 Wire Wire Line
 	14750 2300 14750 2250
-Text Label 13850 5600 3    50   ~ 0
+Text Label 13850 5150 3    50   ~ 0
 Vout
 Wire Wire Line
@@
 F 0 "J3" H 14200 6400 50  0000 C CNN
 F 1 "0.1\" HDR" H 14200 5800 50  0000 C CNN
-F 2 "Connector_PinSocket_2.54mm:PinSocket_2x05_P2.54mm_Vertical" H 14150 6100 50  0001 C CNN
+F 2 "io-master:PinSocket_2x05_P2.54mm_Vertical_AltNumbering" H 14150 6100 50  0001 C CNN
 F 3 "~" H 14150 6100 50  0001 C CNN
 	1    14150 6100
@@
 	13850 6300 13950 6300
 Wire Wire Line
-	13850 4850 13850 5100
+	13850 5050 13850 5400
 Wire Wire Line
 	15150 4000 15350 4000
@@
 P 2500 2500
 F 0 "TP17" V 2500 2700 50  0000 L CNN
-F 1 "TestPoint" V 2604 2572 50  0001 C CNN
+F 1 "DCIN" V 2604 2572 50  0001 C CNN
 F 2 "TestPoint:TestPoint_Pad_D1.0mm" H 2700 2500 50  0001 C CNN
 F 3 "~" H 2700 2500 50  0001 C CNN
@@
 Wire Wire Line
 	3050 3450 3050 2700
-Text Notes 3900 1650 0    50   ~ 0
-INPUT: 4.6-15V
 $Comp
 L Connector:Barrel_Jack_Switch J1
@@
 	2550 3100 2700 3100
 Wire Wire Line
-	13850 5400 13850 6300
+	13850 5700 13850 6300
 Wire Wire Line
 	2550 1700 2550 1850
@@
 L Device:Polyfuse F2
 U 1 1 5E3F2C3B
-P 13850 5250
-F 0 "F2" H 13938 5296 50  0000 L CNN
-F 1 "0.1A" H 13938 5205 50  0000 L CNN
-F 2 "Fuse:Fuse_1206_3216Metric" H 13900 5050 50  0001 L CNN
-F 3 "~" H 13850 5250 50  0001 C CNN
-	1    13850 5250
-	1    0    0    -1
-$EndComp
+P 13850 5550
+F 0 "F2" H 13938 5596 50  0000 L CNN
+F 1 "0.1A" H 13938 5505 50  0000 L CNN
+F 2 "Fuse:Fuse_1206_3216Metric" H 13900 5350 50  0001 L CNN
+F 3 "~" H 13850 5550 50  0001 C CNN
+	1    13850 5550
+	1    0    0    -1
+$EndComp
+Text Notes 3900 1650 0    50   ~ 0
+INPUT: 4.6-15V
+Text Label 3900 1800 0    50   ~ 0
+Vin
+Wire Wire Line
+	3850 1250 2550 1250
+Wire Wire Line
+	6700 1250 3850 1250
+Connection ~ 3850 1250
+Connection ~ 3850 1800
+Wire Wire Line
+	3850 1800 3850 1250
 $EndSCHEMATC
