File: KiCAD/io-master.kicad_pcb (KiCad board)
At the start: 2 copper layers, 0 parts

Commit message: Add v1.0 PCB layout
Parts:
- added C1: 0.47u, Capacitor_SMD:C_0603_1608Metric, F.Cu at (33.2, 75.2)
- added C10: 1u, Capacitor_SMD:C_0603_1608Metric, F.Cu at (79.8, 98.0)
- added C100: 10u, Capacitor_SMD:C_0805_2012Metric, F.Cu at (75.8, 52.5)
- added C101: 1u, Capacitor_SMD:C_0603_1608Metric, F.Cu at (74.2, 49.2)
- added C102: C, Capacitor_SMD:C_0603_1608Metric, F.Cu at (68.0, 45.5)
- added C103: C, Capacitor_SMD:C_0603_1608Metric, F.Cu at (68.0, 38.5)
- added C104: 0.22u, Capacitor_SMD:C_0603_1608Metric, F.Cu at (65.8, 46.2)
- added C105: 82p, Capacitor_SMD:C_0603_1608Metric, F.Cu at (65.5, 39.2)
- added C106: 1u, Capacitor_SMD:C_0603_1608Metric, F.Cu at (74.2, 50.8)
- added C107: 22u, Capacitor_SMD:C_1210_3225Metric, F.Cu at (83.2, 39.5)
- added C108: 22u, Capacitor_SMD:C_1210_3225Metric, F.Cu at (84.5, 45.2)
- added C109: C, Capacitor_SMD:C_1210_3225Metric, F.Cu at (86.8, 39.5)
- added C11: 1u, Capacitor_SMD:C_0603_1608Metric, F.Cu at (50.2, 110.2)
- added C110: C, Capacitor_SMD:C_1210_3225Metric, F.Cu at (88.0, 45.2)
- added C111: 0.1u, Capacitor_SMD:C_0603_1608Metric, F.Cu at (166.0, 114.0)
- added C112: 0.1u, Capacitor_SMD:C_0603_1608Metric, F.Cu at (169.8, 123.8)
- added C113: 0.1u, Capacitor_SMD:C_0603_1608Metric, F.Cu at (166.0, 71.0)
- added C114: 0.1u, Capacitor_SMD:C_0603_1608Metric, F.Cu at (169.8, 80.8)
- added C115: 0.1u, Capacitor_SMD:C_0603_1608Metric, F.Cu at (166.0, 51.2)
- added C116: 0.1u, Capacitor_SMD:C_0603_1608Metric, F.Cu at (169.8, 61.0)
- added C117: 0.1u, Capacitor_SMD:C_0603_1608Metric, F.Cu at (166.0, 94.2)
- added C118: 0.1u, Capacitor_SMD:C_0603_1608Metric, F.Cu at (169.8, 104.0)
- added C12: 20p, Capacitor_SMD:C_0603_1608Metric, F.Cu at (51.2, 101.8)
- added C13: 20p, Capacitor_SMD:C_0603_1608Metric, F.Cu at (51.2, 106.2)
- added C14: 2.2u, Capacitor_SMD:C_0805_2012Metric, F.Cu at (80.2, 89.6)
- added C15: 0.1u, Capacitor_SMD:C_0603_1608Metric, F.Cu at (50.2, 111.8)
- added C16: 0.1u, Capacitor_SMD:C_0603_1608Metric, F.Cu at (53.2, 108.8)
- added C17: 0.1u, Capacitor_SMD:C_0603_1608Metric, F.Cu at (59.0, 113.5)
- added C18: 0.1u, Capacitor_SMD:C_0603_1608Metric, F.Cu at (149.0, 107.0)
- added C19: 0.1u, Capacitor_SMD:C_0603_1608Metric, F.Cu at (65.5, 113.5)
- added C2: 1u, Capacitor_SMD:C_0603_1608Metric, F.Cu at (37.2, 65.8)
- added C20: 0.1u, Capacitor_SMD:C_0603_1608Metric, F.Cu at (70.5, 113.5)
- added C21: 0.1u, Capacitor_SMD:C_0603_1608Metric, F.Cu at (149.0, 64.0)
- added C22: 0.1u, Capacitor_SMD:C_0603_1608Metric, F.Cu at (76.8, 113.5)
- added C23: 0.1u, Capacitor_SMD:C_0603_1608Metric, F.Cu at (79.9, 103.5)
- added C24: 0.1u, Capacitor_SMD:C_0603_1608Metric, F.Cu at (78.5, 89.7)
- added C25: 0.1u, Capacitor_SMD:C_0603_1608Metric, F.Cu at (69.0, 87.0)
- added C26: 0.1u, Capacitor_SMD:C_0603_1608Metric, F.Cu at (64.8, 87.2)
- added C27: 0.1u, Capacitor_SMD:C_0603_1608Metric, F.Cu at (58.0, 87.2)
- added C28: 0.1u, Capacitor_SMD:C_0603_1608Metric, F.Cu at (37.0, 107.8)
- added C29: 4.7u, Capacitor_SMD:C_0805_2012Metric, F.Cu at (52.5, 76.7)
- added C3: 0.1u, Capacitor_SMD:C_0603_1608Metric, F.Cu at (44.0, 42.5)
- added C30: 0.1u, Capacitor_SMD:C_0603_1608Metric, F.Cu at (50.8, 76.5)
- added C31: 0.1u, Capacitor_SMD:C_0603_1608Metric, F.Cu at (44.9, 72.0)
- added C32: 0.1u, Capacitor_SMD:C_0603_1608Metric, F.Cu at (53.8, 67.0)
- added C33: 20p, Capacitor_SMD:C_0603_1608Metric, F.Cu at (54.0, 64.5)
- added C34: 20p, Capacitor_SMD:C_0603_1608Metric, F.Cu at (49.5, 64.5)
- added C35: 0.1u, Capacitor_SMD:C_0603_1608Metric, F.Cu at (53.8, 74.2)
- added C36: 0.1u, Capacitor_SMD:C_0603_1608Metric, F.Cu at (53.8, 68.5)
- added C37: 4.7u, Capacitor_SMD:C_0805_2012Metric, F.Cu at (45.5, 65.0)
- added C38: 0.1u, Capacitor_SMD:C_0603_1608Metric, F.Cu at (45.5, 66.8)
- added C39: 0.1u, Capacitor_SMD:C_0603_1608Metric, F.Cu at (48.0, 66.0)
- added C4: 10u, Capacitor_SMD:C_0805_2012Metric, F.Cu at (46.0, 42.5)
- added C40: C, Capacitor_SMD:C_1210_3225Metric, F.Cu at (99.0, 37.0)
- added C41: 10u, Capacitor_SMD:C_0805_2012Metric, F.Cu at (101.8, 37.0)
- added C42: 0.1u, Capacitor_SMD:C_0603_1608Metric, F.Cu at (115.5, 43.8)
- added C43: 1u, Capacitor_SMD:C_0603_1608Metric, F.Cu at (113.8, 37.0)
- added C44: 33p, Capacitor_SMD:C_0603_1608Metric, F.Cu at (104.8, 45.8)
- added C45: C, Capacitor_SMD:C_1210_3225Metric, F.Cu at (120.0, 40.5)
- added C46: 10u, Capacitor_SMD:C_0805_2012Metric, F.Cu at (117.2, 40.5)
- added C47: 0.1u, Capacitor_SMD:C_0603_1608Metric, F.Cu at (99.8, 95.0)
- added C48: 0.1u, Capacitor_SMD:C_0603_1608Metric, F.Cu at (111.8, 96.0)
- added C49: 0.1u, Capacitor_SMD:C_0603_1608Metric, F.Cu at (111.8, 84.5)
- added C5: 22u, Capacitor_SMD:C_1210_3225Metric, F.Cu at (51.8, 36.8)
- added C50: 0.1u, Capacitor_SMD:C_0603_1608Metric, F.Cu at (127.0, 108.0)
- added C51: 0.1u, Capacitor_SMD:C_0603_1608Metric, F.Cu at (132.2, 87.5)
- added C52: 0.1u, Capacitor_SMD:C_0603_1608Metric, F.Cu at (132.2, 108.0)
- added C53: 0.1u, Capacitor_SMD:C_0603_1608Metric, F.Cu at (126.0, 102.0)
- added C54: 0.1u, Capacitor_SMD:C_0603_1608Metric, F.Cu at (149.0, 112.2)
- added C55: C, Capacitor_SMD:C_0603_1608Metric, F.Cu at (142.8, 106.2)
- added C56: C, Capacitor_SMD:C_0603_1608Metric, F.Cu at (132.2, 100.5)
- added C57: 0.1u, Capacitor_SMD:C_0603_1608Metric, F.Cu at (132.2, 91.5)
- added C58: 0.1u, Capacitor_SMD:C_0603_1608Metric, F.Cu at (132.2, 86.0)
- added C59: C, Capacitor_SMD:C_0603_1608Metric, F.Cu at (142.8, 93.0)
- added C6: 0.1u, Capacitor_SMD:C_0603_1608Metric, F.Cu at (51.8, 34.2)
- added C60: 0.1u, Capacitor_SMD:C_0603_1608Metric, F.Cu at (132.2, 112.5)
- added C61: 0.1u, Capacitor_SMD:C_0603_1608Metric, F.Cu at (142.8, 109.2)
- added C62: 0.1u, Capacitor_SMD:C_0603_1608Metric, F.Cu at (142.8, 99.8)
- added C63: 0.1u, Capacitor_SMD:C_0603_1608Metric, F.Cu at (132.2, 103.5)
- added C64: 10u, Capacitor_SMD:C_0805_2012Metric, F.Cu at (143.0, 82.2)
- added C65: 10u, Capacitor_SMD:C_0805_2012Metric, F.Cu at (132.0, 84.2)
- added C66: 10u, Capacitor_SMD:C_0805_2012Metric, F.Cu at (143.0, 114.0)
- added C67: 10u, Capacitor_SMD:C_0805_2012Metric, F.Cu at (132.0, 118.8)
- added C68: 0.1u, Capacitor_SMD:C_0603_1608Metric, F.Cu at (149.0, 90.5)
- added C69: 0.1u, Capacitor_SMD:C_0603_1608Metric, F.Cu at (149.0, 85.5)
- added C7: 2.2u, Capacitor_SMD:C_0805_2012Metric, F.Cu at (75.0, 113.7)
- added C70: 0.1u, Capacitor_SMD:C_0603_1608Metric, F.Cu at (149.0, 113.8)
- added C71: 0.1u, Capacitor_SMD:C_0603_1608Metric, F.Cu at (149.0, 118.8)
- added C72: 1000p, Capacitor_SMD:C_0603_1608Metric, F.Cu at (159.8, 100.5)
- added C73: 0.1u, Capacitor_SMD:C_0603_1608Metric, F.Cu at (99.8, 71.2)
- added C74: 0.1u, Capacitor_SMD:C_0603_1608Metric, F.Cu at (111.8, 72.2)
- added C75: 0.1u, Capacitor_SMD:C_0603_1608Metric, F.Cu at (111.8, 60.8)
- added C76: 0.1u, Capacitor_SMD:C_0603_1608Metric, F.Cu at (127.0, 65.0)
- added C77: 0.1u, Capacitor_SMD:C_0603_1608Metric, F.Cu at (132.2, 44.5)
- added C78: 0.1u, Capacitor_SMD:C_0603_1608Metric, F.Cu at (132.2, 65.0)
- added C79: 0.1u, Capacitor_SMD:C_0603_1608Metric, F.Cu at (126.0, 59.0)
- added C8: 4.7u, Capacitor_SMD:C_0805_2012Metric, F.Cu at (70.8, 86.8)
- added C80: 0.1u, Capacitor_SMD:C_0603_1608Metric, F.Cu at (149.0, 69.2)
- added C81: C, Capacitor_SMD:C_0603_1608Metric, F.Cu at (142.8, 63.2)
- added C82: C, Capacitor_SMD:C_0603_1608Metric, F.Cu at (132.2, 57.5)
- added C83: 0.1u, Capacitor_SMD:C_0603_1608Metric, F.Cu at (132.2, 48.5)
- added C84: 0.1u, Capacitor_SMD:C_0603_1608Metric, F.Cu at (132.2, 43.0)
- added C85: C, Capacitor_SMD:C_0603_1608Metric, F.Cu at (142.8, 50.0)
- added C86: 0.1u, Capacitor_SMD:C_0603_1608Metric, F.Cu at (132.2, 69.5)
- added C87: 0.1u, Capacitor_SMD:C_0603_1608Metric, F.Cu at (142.8, 66.2)
- added C88: 0.1u, Capacitor_SMD:C_0603_1608Metric, F.Cu at (142.8, 56.8)
- added C89: 0.1u, Capacitor_SMD:C_0603_1608Metric, F.Cu at (132.2, 60.5)
- added C9: 0.1u, Capacitor_SMD:C_0603_1608Metric, F.Cu at (53.0, 98.2)
- added C90: 10u, Capacitor_SMD:C_0805_2012Metric, F.Cu at (143.0, 39.2)
- added C91: 10u, Capacitor_SMD:C_0805_2012Metric, F.Cu at (132.0, 41.2)
- added C92: 10u, Capacitor_SMD:C_0805_2012Metric, F.Cu at (143.0, 71.0)
- added C93: 10u, Capacitor_SMD:C_0805_2012Metric, F.Cu at (132.0, 75.8)
- added C94: 0.1u, Capacitor_SMD:C_0603_1608Metric, F.Cu at (149.0, 47.5)
- added C95: 0.1u, Capacitor_SMD:C_0603_1608Metric, F.Cu at (149.0, 42.5)
- added C96: 0.1u, Capacitor_SMD:C_0603_1608Metric, F.Cu at (149.0, 70.8)
- added C97: 0.1u, Capacitor_SMD:C_0603_1608Metric, F.Cu at (149.0, 75.8)
- added C98: 1000p, Capacitor_SMD:C_0603_1608Metric, F.Cu at (159.8, 57.5)
- added C99: C, Capacitor_SMD:C_1210_3225Metric, F.Cu at (75.8, 55.2)
- added D1: B130L, Diode_SMD:D_SMA, F.Cu at (47.0, 52.0)
- added D10: RGB, io-master:LED_Everlight_19-337C, F.Cu at (48.2, 94.5)
- added D11: YEL/GRN, io-master:LED_Kingbright_APTB1615YSGC, F.Cu at (94.2, 69.5)
- added D12: DDZ5V6ASF, Diode_SMD:D_SOD-323F, F.Cu at (44.2, 70.0)
- added D13: NSR0530HT1G, Diode_SMD:D_SOD-323, F.Cu at (114.8, 34.2)
- added D14: MM3Z9V1ST1G, Diode_SMD:D_SOD-323, F.Cu at (142.8, 98.0)
- added D15: MM3Z9V1ST1G, Diode_SMD:D_SOD-323, F.Cu at (142.8, 103.0)
- added D16: MM3Z15VST1G, Diode_SMD:D_SOD-323, F.Cu at (167.0, 109.8)
- added D17: 1N4148, Diode_SMD:D_SOD-323, F.Cu at (165.5, 119.2)
- added D18: 1N4148, Diode_SMD:D_SOD-323, F.Cu at (165.5, 117.2)
- added D19: RED, LED_SMD:LED_0603_1608Metric, F.Cu at (181.2, 117.2)
- added D2: B130L, Diode_SMD:D_SMA, F.Cu at (43.0, 61.2)
- added D20: MM3Z15VST1G, Diode_SMD:D_SOD-323, F.Cu at (167.0, 107.8)
- added D21: 1N4148, Diode_SMD:D_SOD-323, F.Cu at (165.5, 76.2)
- added D22: 1N4148, Diode_SMD:D_SOD-323, F.Cu at (165.5, 74.2)
- added D23: RED, LED_SMD:LED_0603_1608Metric, F.Cu at (181.2, 74.2)
- added D24: MM3Z15VST1G, Diode_SMD:D_SOD-323, F.Cu at (167.0, 66.8)
- added D25: 1N4148, Diode_SMD:D_SOD-323, F.Cu at (165.5, 56.5)
- added D26: 1N4148, Diode_SMD:D_SOD-323, F.Cu at (165.5, 54.5)
- added D27: RED, LED_SMD:LED_0603_1608Metric, F.Cu at (181.2, 54.5)
- added D28: MM3Z9V1ST1G, Diode_SMD:D_SOD-323, F.Cu at (142.8, 55.0)
- added D29: MM3Z9V1ST1G, Diode_SMD:D_SOD-323, F.Cu at (142.8, 60.0)
- added D3: ORANGE, LED_SMD:LED_0603_1608Metric, F.Cu at (58.5, 47.2)
- added D30: NSR0530HT1G, Diode_SMD:D_SOD-323, F.Cu at (80.5, 38.2)
- added D31: NSR0530HT1G, Diode_SMD:D_SOD-323, F.Cu at (82.5, 49.2)
- added D32: MM3Z15VST1G, Diode_SMD:D_SOD-323, F.Cu at (167.0, 64.8)
- added D33: 1N4148, Diode_SMD:D_SOD-323, F.Cu at (165.5, 99.5)
- added D34: 1N4148, Diode_SMD:D_SOD-323, F.Cu at (165.5, 97.5)
- added D35: RED, LED_SMD:LED_0603_1608Metric, F.Cu at (181.2, 97.5)
- added D36: MM3Z15VST1G, Diode_SMD:D_SOD-323, F.Cu at (167.0, 47.0)
- added D37: MM3Z15VST1G, Diode_SMD:D_SOD-323, F.Cu at (167.0, 45.0)
- added D38: MM3Z15VST1G, Diode_SMD:D_SOD-323, F.Cu at (167.0, 90.0)
- added D39: MM3Z15VST1G, Diode_SMD:D_SOD-323, F.Cu at (167.0, 88.0)
- added D4: BLUE, LED_SMD:LED_0603_1608Metric, F.Cu at (91.8, 37.0)
- added D5: BLUE, LED_SMD:LED_0603_1608Metric, F.Cu at (91.8, 48.8)
- added D6: GREEN, LED_SMD:LED_0603_1608Metric, F.Cu at (123.8, 37.0)
- added D7: YEL/GRN, io-master:LED_Kingbright_APTB1615YSGC, F.Cu at (94.2, 99.2)
- added D8: YEL/GRN, io-master:LED_Kingbright_APTB1615YSGC, F.Cu at (94.2, 90.5)
- added D9: YEL/GRN, io-master:LED_Kingbright_APTB1615YSGC, F.Cu at (94.2, 78.2)
- added F1: 0.5A, Fuse:Fuse_1206_3216Metric, F.Cu at (50.9, 59.8)
- added F2: 0.1A, Fuse:Fuse_1206_3216Metric, F.Cu at (192.2, 67.2)
- added FB1: MZ1608-102Y, Resistor_SMD:R_0603_1608Metric, F.Cu at (53.2, 110.2)
- added H1: M3, MountingHole:MountingHole_3.2mm_M3_Pad, F.Cu at (35.0, 35.0)
- added H2: M3, MountingHole:MountingHole_3.2mm_M3_Pad, F.Cu at (195.0, 35.0)
- added H3: M3, MountingHole:MountingHole_3.2mm_M3_Pad, F.Cu at (35.0, 125.0)
- added H4: M3, MountingHole:MountingHole_3.2mm_M3_Pad, F.Cu at (195.0, 125.0)
- added J1: 54-00166, io-master:BarrelJack_Tensility_54-00166_Horizontal, F.Cu at (43.0, 50.0)
- added J2: 10118193, io-master:USB_Micro-B_Amphenol_10118193-0001LF_Horizontal, F.Cu at (31.5, 70.0)
- added J3: 0.1" HDR, io-master:PinSocket_2x05_P2.54mm_Vertical_AltNumbering, F.Cu at (191.0, 82.1)
- added J4: 0.1" HDR, Connector_PinSocket_2.54mm:PinSocket_2x05_P2.54mm_Vertical, F.Cu at (74.2, 75.8)
- added L1: 82u, io-master:L_Bourns_SRF0703, F.Cu at (107.2, 37.0)
- added L2: 10u, io-master:L_Abracon_ASPI-0418FS, F.Cu at (76.8, 36.8)
- added L3: 15u, Inductor_SMD:L_Taiyo-Yuden_NR-50xx, F.Cu at (80.0, 45.2)
- added Q1: Q_NPN_BCE, Package_TO_SOT_SMD:SOT-323_SC-70, F.Cu at (177.8, 40.2)
- added Q10: DMN63D8LDW, Package_TO_SOT_SMD:SOT-363_SC-70-6, F.Cu at (157.0, 101.2)
- added Q11: DMN63D8LDW, Package_TO_SOT_SMD:SOT-363_SC-70-6, F.Cu at (173.8, 111.2)
- added Q12: MMBT3906, Package_TO_SOT_SMD:SOT-323_SC-70, F.Cu at (178.2, 119.0)
- added Q13: DMN63D8LDW, Package_TO_SOT_SMD:SOT-363_SC-70-6, F.Cu at (173.8, 68.2)
- added Q14: MMBT3906, Package_TO_SOT_SMD:SOT-323_SC-70, F.Cu at (178.2, 76.0)
- added Q15: DMN63D8LDW, Package_TO_SOT_SMD:SOT-363_SC-70-6, F.Cu at (173.8, 48.5)
- added Q16: MMBT3906, Package_TO_SOT_SMD:SOT-323_SC-70, F.Cu at (178.2, 56.2)
- added Q17: MMBT3904, Package_TO_SOT_SMD:SOT-323_SC-70, F.Cu at (159.5, 73.8)
- added Q18: MMBT3906, Package_TO_SOT_SMD:SOT-323_SC-70, F.Cu at (154.5, 73.8)
- added Q19: DMG1029SV, Package_TO_SOT_SMD:SOT-563, F.Cu at (157.0, 71.0)
- added Q2: Q_NPN_BCE, Package_TO_SOT_SMD:SOT-323_SC-70, F.Cu at (110.5, 114.8)
- added Q20: MMBT3904, Package_TO_SOT_SMD:SOT-323_SC-70, F.Cu at (159.5, 43.0)
- added Q21: MMBT3906, Package_TO_SOT_SMD:SOT-323_SC-70, F.Cu at (154.5, 43.0)
- added Q22: DMG1029SV, Package_TO_SOT_SMD:SOT-563, F.Cu at (157.0, 45.8)
- added Q23: MMBT3904, Package_TO_SOT_SMD:SOT-323_SC-70, F.Cu at (155.5, 61.2)
- added Q24: DMN63D8LDW, Package_TO_SOT_SMD:SOT-363_SC-70-6, F.Cu at (157.0, 58.2)
- added Q25: DMN63D8LDW, Package_TO_SOT_SMD:SOT-363_SC-70-6, F.Cu at (173.8, 91.5)
- added Q26: MMBT3906, Package_TO_SOT_SMD:SOT-323_SC-70, F.Cu at (178.2, 99.2)
- added Q27: DMP3099L, Package_TO_SOT_SMD:SOT-23, F.Cu at (37.5, 61.2)
- added Q3: MMBT3904, Package_TO_SOT_SMD:SOT-323_SC-70, F.Cu at (159.5, 116.8)
- added Q4: MMBT3906, Package_TO_SOT_SMD:SOT-323_SC-70, F.Cu at (154.5, 116.8)
- added Q5: DMG1029SV, Package_TO_SOT_SMD:SOT-563, F.Cu at (157.0, 114.0)
- added Q6: MMBT3904, Package_TO_SOT_SMD:SOT-323_SC-70, F.Cu at (159.5, 86.0)
- added Q7: MMBT3906, Package_TO_SOT_SMD:SOT-323_SC-70, F.Cu at (154.5, 86.0)
- added Q8: DMG1029SV, Package_TO_SOT_SMD:SOT-563, F.Cu at (157.0, 88.8)
- added Q9: MMBT3904, Package_TO_SOT_SMD:SOT-323_SC-70, F.Cu at (155.5, 104.2)
- added R1: R, Resistor_SMD:R_0603_1608Metric, F.Cu at (170.2, 39.2)
- added R10: 100K, Resistor_SMD:R_0603_1608Metric, F.Cu at (87.0, 99.2)
- added R100: 10K, Resistor_SMD:R_0603_1608Metric, F.Cu at (159.8, 83.0)
- added R101: 10K, Resistor_SMD:R_0603_1608Metric, F.Cu at (154.2, 83.0)
- added R102: 100K, Resistor_SMD:R_0603_1608Metric, F.Cu at (132.2, 81.0)
- added R103: 100K, Resistor_SMD:R_0603_1608Metric, F.Cu at (132.2, 117.0)
- added R104: 100K, Resistor_SMD:R_0603_1608Metric, F.Cu at (160.0, 89.0)
- added R105: 100K, Resistor_SMD:R_0603_1608Metric, F.Cu at (154.0, 89.0)
- added R106: 100K, Resistor_SMD:R_0603_1608Metric, F.Cu at (132.2, 82.5)
- added R107: 100K, Resistor_SMD:R_0603_1608Metric, F.Cu at (132.2, 115.5)
- added R108: 10K, Resistor_SMD:R_0603_1608Metric, F.Cu at (155.2, 90.5)
- added R109: 10K, Resistor_SMD:R_0603_1608Metric, F.Cu at (158.8, 90.5)
- added R11: 1K, Resistor_SMD:R_0603_1608Metric, F.Cu at (94.2, 97.5)
- added R110: 0, Resistor_SMD:R_0603_1608Metric, F.Cu at (142.8, 87.0)
- added R111: 0, Resistor_SMD:R_0603_1608Metric, F.Cu at (142.8, 118.8)
- added R112: 100K, Resistor_SMD:R_0603_1608Metric, F.Cu at (142.8, 85.5)
- added R113: 100K, Resistor_SMD:R_0603_1608Metric, F.Cu at (142.8, 115.8)
- added R114: 0, Resistor_SMD:R_0603_1608Metric, F.Cu at (142.8, 84.0)
- added R115: 0, Resistor_SMD:R_0603_1608Metric, F.Cu at (142.8, 117.2)
- added R116: 10K, Resistor_SMD:R_0603_1608Metric, F.Cu at (153.2, 102.0)
- added R117: 100K, Resistor_SMD:R_0603_1608Metric, F.Cu at (153.2, 100.5)
- added R118: 100K, Resistor_SMD:R_0603_1608Metric, F.Cu at (159.8, 102.0)
- added R119: 120, Resistor_SMD:R_0805_2012Metric, F.Cu at (156.0, 108.8)
- added R12: 100K, Resistor_SMD:R_0603_1608Metric, F.Cu at (87.0, 90.5)
- added R120: 120, Resistor_SMD:R_0805_2012Metric, F.Cu at (156.0, 94.0)
- added R121: 120, Resistor_SMD:R_0805_2012Metric, F.Cu at (158.0, 108.8)
- added R122: 120, Resistor_SMD:R_0805_2012Metric, F.Cu at (158.0, 94.0)
- added R123: 2, Resistor_SMD:R_0603_1608Metric, F.Cu at (170.5, 111.2)
- added R124: 10K, Resistor_SMD:R_0603_1608Metric, F.Cu at (171.2, 113.5)
- added R125: 10K, Resistor_SMD:R_0603_1608Metric, F.Cu at (169.8, 113.5)
- added R126: 100K, Resistor_SMD:R_0603_1608Metric, F.Cu at (166.0, 112.5)
- added R127: 100K, Resistor_SMD:R_0603_1608Metric, F.Cu at (174.5, 114.2)
- added R128: 100K, Resistor_SMD:R_0603_1608Metric, F.Cu at (174.5, 115.8)
- added R129: 100K, Resistor_SMD:R_0603_1608Metric, F.Cu at (165.8, 121.0)
- added R13: 1K, Resistor_SMD:R_0603_1608Metric, F.Cu at (94.2, 101.0)
- added R130: 100K, Resistor_SMD:R_0603_1608Metric, F.Cu at (166.0, 115.5)
- added R131: 100K, Resistor_SMD:R_0603_1608Metric, F.Cu at (165.8, 122.5)
- added R132: 100K, Resistor_SMD:R_0603_1608Metric, F.Cu at (165.8, 124.0)
- added R133: 100K, Resistor_SMD:R_0603_1608Metric, F.Cu at (174.5, 122.5)
- added R134: 6.8K, Resistor_SMD:R_0603_1608Metric, F.Cu at (174.5, 121.0)
- added R135: 100K, Resistor_SMD:R_0603_1608Metric, F.Cu at (173.8, 109.2)
- added R136: 10K, Resistor_SMD:R_0603_1608Metric, F.Cu at (174.5, 124.0)
- added R137: 10K, Resistor_SMD:R_0603_1608Metric, F.Cu at (174.5, 117.2)
- added R138: 2, Resistor_SMD:R_0603_1608Metric, F.Cu at (170.5, 68.2)
- added R139: 10K, Resistor_SMD:R_0603_1608Metric, F.Cu at (171.2, 70.5)
- added R14: 100K, Resistor_SMD:R_0603_1608Metric, F.Cu at (87.0, 97.5)
- added R140: 10K, Resistor_SMD:R_0603_1608Metric, F.Cu at (169.8, 70.5)
- added R141: 100K, Resistor_SMD:R_0603_1608Metric, F.Cu at (166.0, 69.5)
- added R142: 100K, Resistor_SMD:R_0603_1608Metric, F.Cu at (174.5, 71.2)
- added R143: 100K, Resistor_SMD:R_0603_1608Metric, F.Cu at (174.5, 72.8)
- added R144: 100K, Resistor_SMD:R_0603_1608Metric, F.Cu at (165.8, 78.0)
- added R145: 100K, Resistor_SMD:R_0603_1608Metric, F.Cu at (166.0, 72.5)
- added R146: 100K, Resistor_SMD:R_0603_1608Metric, F.Cu at (165.8, 79.5)
- added R147: 100K, Resistor_SMD:R_0603_1608Metric, F.Cu at (165.8, 81.0)
- added R148: 100K, Resistor_SMD:R_0603_1608Metric, F.Cu at (174.5, 79.5)
- added R149: 6.8K, Resistor_SMD:R_0603_1608Metric, F.Cu at (174.5, 78.0)
- added R15: 100K, Resistor_SMD:R_0603_1608Metric, F.Cu at (87.0, 88.8)
- added R150: 100K, Resistor_SMD:R_0603_1608Metric, F.Cu at (173.8, 66.2)
- added R151: 10K, Resistor_SMD:R_0603_1608Metric, F.Cu at (174.5, 81.0)
- added R152: 10K, Resistor_SMD:R_0603_1608Metric, F.Cu at (174.5, 74.2)
- added R153: 2, Resistor_SMD:R_0603_1608Metric, F.Cu at (170.5, 48.5)
- added R154: 10K, Resistor_SMD:R_0603_1608Metric, F.Cu at (171.2, 50.8)
- added R155: 10K, Resistor_SMD:R_0603_1608Metric, F.Cu at (169.8, 50.8)
- added R156: 100K, Resistor_SMD:R_0603_1608Metric, F.Cu at (166.0, 49.8)
- added R157: 100K, Resistor_SMD:R_0603_1608Metric, F.Cu at (174.5, 51.5)
- added R158: 100K, Resistor_SMD:R_0603_1608Metric, F.Cu at (174.5, 53.0)
- added R159: 100K, Resistor_SMD:R_0603_1608Metric, F.Cu at (165.8, 58.2)
- added R16: 4.7K, Resistor_SMD:R_0603_1608Metric, F.Cu at (79.8, 95.0)
- added R160: 100K, Resistor_SMD:R_0603_1608Metric, F.Cu at (166.0, 52.8)
- added R161: 100K, Resistor_SMD:R_0603_1608Metric, F.Cu at (165.8, 59.8)
- added R162: 100K, Resistor_SMD:R_0603_1608Metric, F.Cu at (165.8, 61.2)
- added R163: 100K, Resistor_SMD:R_0603_1608Metric, F.Cu at (174.5, 59.8)
- added R164: 6.8K, Resistor_SMD:R_0603_1608Metric, F.Cu at (174.5, 58.2)
- added R165: 100K, Resistor_SMD:R_0603_1608Metric, F.Cu at (173.8, 46.5)
- added R166: 10K, Resistor_SMD:R_0603_1608Metric, F.Cu at (174.5, 61.2)
- added R167: 10K, Resistor_SMD:R_0603_1608Metric, F.Cu at (174.5, 54.5)
- added R168: 100K, Resistor_SMD:R_0603_1608Metric, F.Cu at (108.0, 74.5)
- added R169: 100K, Resistor_SMD:R_0603_1608Metric, F.Cu at (108.0, 73.0)
- added R17: 100K, Resistor_SMD:R_0603_1608Metric, F.Cu at (89.2, 95.8)
- added R170: 100K, Resistor_SMD:R_0603_1608Metric, F.Cu at (115.5, 74.5)
- added R171: 100K, Resistor_SMD:R_0603_1608Metric, F.Cu at (115.5, 73.0)
- added R172: 100K, Resistor_SMD:R_0603_1608Metric, F.Cu at (115.5, 58.5)
- added R173: 100K, Resistor_SMD:R_0603_1608Metric, F.Cu at (115.5, 60.0)
- added R174: 100K, Resistor_SMD:R_0603_1608Metric, F.Cu at (108.0, 58.5)
- added R175: 100K, Resistor_SMD:R_0603_1608Metric, F.Cu at (108.0, 60.0)
- added R176: 110K, Resistor_SMD:R_0603_1608Metric, F.Cu at (107.5, 69.8)
- added R177: 110K, Resistor_SMD:R_0603_1608Metric, F.Cu at (110.2, 72.2)
- added R178: 110K, Resistor_SMD:R_0603_1608Metric, F.Cu at (116.2, 68.2)
- added R179: 110K, Resistor_SMD:R_0603_1608Metric, F.Cu at (113.2, 72.2)
- added R18: 4.7K, Resistor_SMD:R_0603_1608Metric, F.Cu at (79.8, 96.5)
- added R180: 110K, Resistor_SMD:R_0603_1608Metric, F.Cu at (116.2, 64.8)
- added R181: 110K, Resistor_SMD:R_0603_1608Metric, F.Cu at (113.2, 60.8)
- added R182: 110K, Resistor_SMD:R_0603_1608Metric, F.Cu at (107.2, 64.8)
- added R183: 110K, Resistor_SMD:R_0603_1608Metric, F.Cu at (110.2, 60.8)
- added R184: 1M, Resistor_SMD:R_0603_1608Metric, F.Cu at (108.0, 71.5)
- added R185: 1M, Resistor_SMD:R_0603_1608Metric, F.Cu at (115.5, 71.5)
- added R186: 1M, Resistor_SMD:R_0603_1608Metric, F.Cu at (115.5, 61.5)
- added R187: 1M, Resistor_SMD:R_0603_1608Metric, F.Cu at (108.0, 61.5)
- added R188: 1M, Resistor_SMD:R_0603_1608Metric, F.Cu at (107.5, 68.2)
- added R189: 1M, Resistor_SMD:R_0603_1608Metric, F.Cu at (116.2, 69.8)
- added R19: 1K, Resistor_SMD:R_0603_1608Metric, F.Cu at (94.2, 88.8)
- added R190: 1M, Resistor_SMD:R_0603_1608Metric, F.Cu at (116.2, 63.2)
- added R191: 1M, Resistor_SMD:R_0603_1608Metric, F.Cu at (107.2, 63.2)
- added R192: 100K, Resistor_SMD:R_0603_1608Metric, F.Cu at (132.2, 50.0)
- added R193: 100K, Resistor_SMD:R_0603_1608Metric, F.Cu at (132.2, 51.5)
- added R194: 110K, Resistor_SMD:R_0603_1608Metric, F.Cu at (142.8, 64.8)
- added R195: R, Resistor_SMD:R_0603_1608Metric, F.Cu at (139.8, 63.2)
- added R196: R, Resistor_SMD:R_0603_1608Metric, F.Cu at (132.2, 54.5)
- added R197: 1M, Resistor_SMD:R_0603_1608Metric, F.Cu at (132.2, 62.0)
- added R198: 110K, Resistor_SMD:R_0603_1608Metric, F.Cu at (132.2, 63.5)
- added R199: 1M, Resistor_SMD:R_0603_1608Metric, F.Cu at (142.8, 68.2)
- added R2: R, Resistor_SMD:R_0603_1608Metric, F.Cu at (170.2, 41.2)
- added R20: 100K, Resistor_SMD:R_0603_1608Metric, F.Cu at (89.2, 104.5)
- added R200: 110K, Resistor_SMD:R_0603_1608Metric, F.Cu at (142.8, 51.5)
- added R201: 100K, Resistor_SMD:R_0603_1608Metric, F.Cu at (142.8, 58.2)
- added R202: 1M, Resistor_SMD:R_0603_1608Metric, F.Cu at (142.8, 45.5)
- added R203: 110K, Resistor_SMD:R_0603_1608Metric, F.Cu at (142.8, 47.0)
- added R204: 47K, Resistor_SMD:R_0603_1608Metric, F.Cu at (132.2, 56.0)
- added R205: 1M, Resistor_SMD:R_0603_1608Metric, F.Cu at (142.8, 48.5)
- added R206: 100K, Resistor_SMD:R_0603_1608Metric, F.Cu at (127.0, 69.5)
- added R207: 100K, Resistor_SMD:R_0603_1608Metric, F.Cu at (127.0, 71.0)
- added R208: 47K, Resistor_SMD:R_0603_1608Metric, F.Cu at (132.2, 59.0)
- added R209: R, Resistor_SMD:R_0603_1608Metric, F.Cu at (139.8, 51.5)
- added R21: 100K, Resistor_SMD:R_0603_1608Metric, F.Cu at (89.2, 102.8)
- added R210: 47K, Resistor_SMD:R_0603_1608Metric, F.Cu at (142.8, 53.2)
- added R211: 47K, Resistor_SMD:R_0603_1608Metric, F.Cu at (142.8, 61.8)
- added R212: 10K, Resistor_SMD:R_0603_1608Metric, F.Cu at (159.8, 76.8)
- added R213: 10K, Resistor_SMD:R_0603_1608Metric, F.Cu at (154.0, 76.8)
- added R214: 100K, Resistor_SMD:R_0603_1608Metric, F.Cu at (160.0, 70.8)
- added R215: 100K, Resistor_SMD:R_0603_1608Metric, F.Cu at (154.0, 70.8)
- added R216: 10K, Resistor_SMD:R_0603_1608Metric, F.Cu at (155.2, 69.2)
- added R217: 10K, Resistor_SMD:R_0603_1608Metric, F.Cu at (158.8, 69.2)
- added R218: 10K, Resistor_SMD:R_0603_1608Metric, F.Cu at (159.8, 40.0)
- added R219: 10K, Resistor_SMD:R_0603_1608Metric, F.Cu at (154.2, 40.0)
- added R22: 1K, Resistor_SMD:R_0603_1608Metric, F.Cu at (94.2, 92.2)
- added R220: 100K, Resistor_SMD:R_0603_1608Metric, F.Cu at (132.2, 38.0)
- added R221: 100K, Resistor_SMD:R_0603_1608Metric, F.Cu at (132.2, 74.0)
- added R222: 100K, Resistor_SMD:R_0603_1608Metric, F.Cu at (160.0, 46.0)
- added R223: 100K, Resistor_SMD:R_0603_1608Metric, F.Cu at (154.0, 46.0)
- added R224: 100K, Resistor_SMD:R_0603_1608Metric, F.Cu at (132.2, 39.5)
- added R225: 100K, Resistor_SMD:R_0603_1608Metric, F.Cu at (132.2, 72.5)
- added R226: 10K, Resistor_SMD:R_0603_1608Metric, F.Cu at (155.2, 47.5)
- added R227: 10K, Resistor_SMD:R_0603_1608Metric, F.Cu at (158.8, 47.5)
- added R228: 0, Resistor_SMD:R_0603_1608Metric, F.Cu at (142.8, 43.9)
- added R229: 0, Resistor_SMD:R_0603_1608Metric, F.Cu at (142.8, 75.8)
- added R23: 100K, Resistor_SMD:R_0603_1608Metric, F.Cu at (89.2, 85.2)
- added R230: 100K, Resistor_SMD:R_0603_1608Metric, F.Cu at (142.8, 42.5)
- added R231: 100K, Resistor_SMD:R_0603_1608Metric, F.Cu at (142.8, 72.8)
- added R232: 0, Resistor_SMD:R_0603_1608Metric, F.Cu at (142.8, 41.0)
- added R233: 0, Resistor_SMD:R_0603_1608Metric, F.Cu at (142.8, 74.2)
- added R234: 10K, Resistor_SMD:R_0603_1608Metric, F.Cu at (153.2, 59.0)
- added R235: 100K, Resistor_SMD:R_0603_1608Metric, F.Cu at (153.2, 57.5)
- added R236: 100K, Resistor_SMD:R_0603_1608Metric, F.Cu at (159.8, 59.0)
- added R237: 120, Resistor_SMD:R_0805_2012Metric, F.Cu at (156.0, 65.8)
- added R238: 120, Resistor_SMD:R_0805_2012Metric, F.Cu at (156.0, 51.0)
- added R239: 120, Resistor_SMD:R_0805_2012Metric, F.Cu at (158.0, 65.8)
- added R24: 100K, Resistor_SMD:R_0603_1608Metric, F.Cu at (89.2, 87.0)
- added R240: 120, Resistor_SMD:R_0805_2012Metric, F.Cu at (158.0, 51.0)
- added R241: 5.36K, Resistor_SMD:R_0603_1608Metric, F.Cu at (68.0, 47.0)
- added R242: 390K, Resistor_SMD:R_0603_1608Metric, F.Cu at (68.0, 40.0)
- added R243: 2.43M, Resistor_SMD:R_0603_1608Metric, F.Cu at (69.0, 35.5)
- added R244: 137K, Resistor_SMD:R_0603_1608Metric, F.Cu at (69.0, 37.0)
- added R245: 118K, Resistor_SMD:R_0603_1608Metric, F.Cu at (71.5, 49.8)
- added R246: 2.32M, Resistor_SMD:R_0603_1608Metric, F.Cu at (70.0, 49.8)
- added R247: 2, Resistor_SMD:R_0603_1608Metric, F.Cu at (170.5, 91.5)
- added R248: 10K, Resistor_SMD:R_0603_1608Metric, F.Cu at (171.2, 93.8)
- added R249: 10K, Resistor_SMD:R_0603_1608Metric, F.Cu at (169.8, 93.8)
- added R25: 100K, Resistor_SMD:R_0603_1608Metric, F.Cu at (87.0, 78.2)
- added R250: 100K, Resistor_SMD:R_0603_1608Metric, F.Cu at (166.0, 92.8)
- added R251: 100K, Resistor_SMD:R_0603_1608Metric, F.Cu at (174.5, 94.5)
- added R252: 100K, Resistor_SMD:R_0603_1608Metric, F.Cu at (174.5, 96.0)
- added R253: 100K, Resistor_SMD:R_0603_1608Metric, F.Cu at (165.8, 101.2)
- added R254: 100K, Resistor_SMD:R_0603_1608Metric, F.Cu at (166.0, 95.8)
- added R255: 100K, Resistor_SMD:R_0603_1608Metric, F.Cu at (165.8, 102.8)
- added R256: 100K, Resistor_SMD:R_0603_1608Metric, F.Cu at (165.8, 104.2)
- added R257: 100K, Resistor_SMD:R_0603_1608Metric, F.Cu at (174.5, 102.8)
- added R258: 6.8K, Resistor_SMD:R_0603_1608Metric, F.Cu at (174.5, 101.2)
- added R259: 100K, Resistor_SMD:R_0603_1608Metric, F.Cu at (173.8, 89.5)
- added R26: 100K, Resistor_SMD:R_0603_1608Metric, F.Cu at (89.2, 94.0)
- added R260: 10K, Resistor_SMD:R_0603_1608Metric, F.Cu at (174.5, 104.2)
- added R261: 10K, Resistor_SMD:R_0603_1608Metric, F.Cu at (174.5, 97.5)
- added R262: 100K, Resistor_SMD:R_0603_1608Metric, F.Cu at (37.2, 58.5)
- added R27: 330, Resistor_SMD:R_0603_1608Metric, F.Cu at (51.2, 94.5)
- added R28: 330, Resistor_SMD:R_0603_1608Metric, F.Cu at (51.2, 96.0)
- added R29: 330, Resistor_SMD:R_0603_1608Metric, F.Cu at (51.2, 93.0)
- added R3: R, Resistor_SMD:R_0603_1608Metric, F.Cu at (107.5, 114.5)
- added R30: 1K, Resistor_SMD:R_0603_1608Metric, F.Cu at (94.2, 76.5)
- added R31: 100K, Resistor_SMD:R_0603_1608Metric, F.Cu at (87.0, 69.5)
- added R32: 100K, Resistor_SMD:R_0603_1608Metric, F.Cu at (89.2, 81.8)
- added R33: 1K, Resistor_SMD:R_0603_1608Metric, F.Cu at (94.2, 80.0)
- added R34: 100K, Resistor_SMD:R_0603_1608Metric, F.Cu at (87.0, 76.5)
- added R35: 100K, Resistor_SMD:R_0603_1608Metric, F.Cu at (89.2, 66.0)
- added R36: 100K, Resistor_SMD:R_0603_1608Metric, F.Cu at (87.0, 67.8)
- added R37: 100K, Resistor_SMD:R_0603_1608Metric, F.Cu at (89.2, 74.8)
- added R38: 100K, Resistor_SMD:R_0603_1608Metric, F.Cu at (89.2, 73.0)
- added R39: 1K, Resistor_SMD:R_0603_1608Metric, F.Cu at (94.2, 67.8)
- added R4: R, Resistor_SMD:R_0603_1608Metric, F.Cu at (105.5, 114.5)
- added R40: 1K, Resistor_SMD:R_0603_1608Metric, F.Cu at (94.2, 71.2)
- added R41: 100K, Resistor_SMD:R_0603_1608Metric, F.Cu at (89.2, 83.5)
- added R42: 100K, Resistor_SMD:R_0603_1608Metric, F.Cu at (89.2, 64.2)
- added R43: 10K, Resistor_SMD:R_0603_1608Metric, F.Cu at (46.0, 82.2)
- added R44: 820, Resistor_SMD:R_0603_1608Metric, F.Cu at (40.0, 68.2)
- added R45: 12K, Resistor_SMD:R_0603_1608Metric, F.Cu at (45.5, 68.2)
- added R46: 1M, Resistor_SMD:R_0603_1608Metric, F.Cu at (50.2, 66.8)
- added R47: 220K, Resistor_SMD:R_0603_1608Metric, F.Cu at (106.5, 42.8)
- added R48: 110K, Resistor_SMD:R_0603_1608Metric, F.Cu at (106.5, 45.8)
- added R49: 10K, Resistor_SMD:R_0603_1608Metric, F.Cu at (103.0, 45.8)
- added R5: 1K, Resistor_SMD:R_0603_1608Metric, F.Cu at (60.2, 47.2)
- added R50: 100K, Resistor_SMD:R_0603_1608Metric, F.Cu at (108.0, 98.2)
- added R51: 100K, Resistor_SMD:R_0603_1608Metric, F.Cu at (108.0, 96.8)
- added R52: 100K, Resistor_SMD:R_0603_1608Metric, F.Cu at (115.5, 98.2)
- added R53: 100K, Resistor_SMD:R_0603_1608Metric, F.Cu at (115.5, 96.8)
- added R54: 100K, Resistor_SMD:R_0603_1608Metric, F.Cu at (115.5, 82.2)
- added R55: 100K, Resistor_SMD:R_0603_1608Metric, F.Cu at (115.5, 83.8)
- added R56: 100K, Resistor_SMD:R_0603_1608Metric, F.Cu at (108.0, 82.2)
- added R57: 100K, Resistor_SMD:R_0603_1608Metric, F.Cu at (108.0, 83.8)
- added R58: 110K, Resistor_SMD:R_0603_1608Metric, F.Cu at (107.2, 92.0)
- added R59: 110K, Resistor_SMD:R_0603_1608Metric, F.Cu at (110.2, 96.0)
- added R6: 10K, Resistor_SMD:R_0603_1608Metric, F.Cu at (91.8, 38.5)
- added R60: 110K, Resistor_SMD:R_0603_1608Metric, F.Cu at (116.2, 92.0)
- added R61: 110K, Resistor_SMD:R_0603_1608Metric, F.Cu at (113.2, 96.0)
- added R62: 110K, Resistor_SMD:R_0603_1608Metric, F.Cu at (116.2, 88.5)
- added R63: 110K, Resistor_SMD:R_0603_1608Metric, F.Cu at (113.2, 84.5)
- added R64: 110K, Resistor_SMD:R_0603_1608Metric, F.Cu at (107.2, 88.5)
- added R65: 110K, Resistor_SMD:R_0603_1608Metric, F.Cu at (110.2, 84.5)
- added R66: 1M, Resistor_SMD:R_0603_1608Metric, F.Cu at (108.0, 95.2)
- added R67: 1M, Resistor_SMD:R_0603_1608Metric, F.Cu at (115.5, 95.2)
- added R68: 1M, Resistor_SMD:R_0603_1608Metric, F.Cu at (115.5, 85.2)
- added R69: 1M, Resistor_SMD:R_0603_1608Metric, F.Cu at (108.0, 85.2)
- added R7: 10K, Resistor_SMD:R_0603_1608Metric, F.Cu at (91.8, 47.2)
- added R70: 1M, Resistor_SMD:R_0603_1608Metric, F.Cu at (107.2, 93.5)
- added R71: 1M, Resistor_SMD:R_0603_1608Metric, F.Cu at (116.2, 93.5)
- added R72: 1M, Resistor_SMD:R_0603_1608Metric, F.Cu at (116.2, 87.0)
- added R73: 1M, Resistor_SMD:R_0603_1608Metric, F.Cu at (107.2, 87.0)
- added R74: 100K, Resistor_SMD:R_0603_1608Metric, F.Cu at (132.2, 93.0)
- added R75: 100K, Resistor_SMD:R_0603_1608Metric, F.Cu at (132.2, 94.5)
- added R76: 110K, Resistor_SMD:R_0603_1608Metric, F.Cu at (142.8, 107.8)
- added R77: R, Resistor_SMD:R_0603_1608Metric, F.Cu at (139.8, 106.2)
- added R78: R, Resistor_SMD:R_0603_1608Metric, F.Cu at (132.2, 97.5)
- added R79: 1M, Resistor_SMD:R_0603_1608Metric, F.Cu at (132.2, 105.0)
- added R8: 4.7K, Resistor_SMD:R_0603_1608Metric, F.Cu at (123.8, 38.8)
- added R80: 110K, Resistor_SMD:R_0603_1608Metric, F.Cu at (132.2, 106.5)
- added R81: 1M, Resistor_SMD:R_0603_1608Metric, F.Cu at (142.8, 111.2)
- added R82: 110K, Resistor_SMD:R_0603_1608Metric, F.Cu at (142.8, 94.5)
- added R83: 100K, Resistor_SMD:R_0603_1608Metric, F.Cu at (142.8, 101.2)
- added R84: 1M, Resistor_SMD:R_0603_1608Metric, F.Cu at (142.8, 88.5)
- added R85: 110K, Resistor_SMD:R_0603_1608Metric, F.Cu at (142.8, 90.0)
- added R86: 47K, Resistor_SMD:R_0603_1608Metric, F.Cu at (132.2, 99.0)
- added R87: 1M, Resistor_SMD:R_0603_1608Metric, F.Cu at (142.8, 91.5)
- added R88: 100K, Resistor_SMD:R_0603_1608Metric, F.Cu at (127.0, 112.5)
- added R89: 100K, Resistor_SMD:R_0603_1608Metric, F.Cu at (127.0, 114.0)
- added R9: R, Resistor_SMD:R_0603_1608Metric, F.Cu at (53.2, 104.0)
- added R90: 47K, Resistor_SMD:R_0603_1608Metric, F.Cu at (132.2, 102.0)
- added R91: R, Resistor_SMD:R_0603_1608Metric, F.Cu at (139.8, 94.5)
- added R92: 47K, Resistor_SMD:R_0603_1608Metric, F.Cu at (142.8, 96.2)
- added R93: 47K, Resistor_SMD:R_0603_1608Metric, F.Cu at (142.8, 104.8)
- added R94: 10K, Resistor_SMD:R_0603_1608Metric, F.Cu at (159.8, 119.8)
- added R95: 10K, Resistor_SMD:R_0603_1608Metric, F.Cu at (154.0, 119.8)
- added R96: 100K, Resistor_SMD:R_0603_1608Metric, F.Cu at (160.0, 113.8)
- added R97: 100K, Resistor_SMD:R_0603_1608Metric, F.Cu at (154.0, 113.8)
- added R98: 10K, Resistor_SMD:R_0603_1608Metric, F.Cu at (155.2, 112.2)
- added R99: 10K, Resistor_SMD:R_0603_1608Metric, F.Cu at (158.8, 112.2)
- added REF**: Symbol_Barrel_Polarity, Symbol:Symbol_Barrel_Polarity, F.Cu at (37.8, 43.8)
- added REF**: OSHW-Logo_5.7x6mm_Copper, Symbol:OSHW-Logo_5.7x6mm_Copper, F.Cu at (98.0, 124.0)
- added REF**: OSHW-Logo_5.7x6mm_Mask, io-master:OSHW-Logo_5.7x6mm_Mask, F.Cu at (98.0, 124.0)
- added SW1: JS202011SCQN, io-master:SW_DPDT_CK_JS202011SCQN, F.Cu at (40.0, 82.2)
- added SW2: EVQ-Q2B03W, Button_Switch_SMD:SW_SPST_EVQQ2, F.Cu at (37.0, 101.8)
- added TP1: TestPoint, TestPoint:TestPoint_Pad_D1.0mm, F.Cu at (168.0, 39.2)
- added TP10: TestPoint, TestPoint:TestPoint_Pad_D1.0mm, F.Cu at (107.5, 116.8)
- added TP100: TRIS8, TestPoint:TestPoint_Pad_D1.0mm, F.Cu at (88.0, 109.2)
- added TP101: SCL, TestPoint:TestPoint_Pad_D1.0mm, F.Cu at (85.0, 117.0)
- added TP102: SDA, TestPoint:TestPoint_Pad_D1.0mm, F.Cu at (86.2, 118.0)
- added TP103: VSET, TestPoint:TestPoint_Pad_D1.0mm, F.Cu at (103.0, 50.8)
- added TP104: PD1, TestPoint:TestPoint_Pad_D1.0mm, F.Cu at (91.8, 102.8)
- added TP105: PD2, TestPoint:TestPoint_Pad_D1.0mm, F.Cu at (91.8, 87.0)
- added TP106: PD3, TestPoint:TestPoint_Pad_D1.0mm, F.Cu at (91.8, 81.8)
- added TP107: PD4, TestPoint:TestPoint_Pad_D1.0mm, F.Cu at (91.8, 66.0)
- added TP108: SW, TestPoint:TestPoint_Pad_D1.0mm, F.Cu at (113.8, 41.0)
- added TP109: TestPoint, TestPoint:TestPoint_Pad_D1.0mm, F.Cu at (112.2, 34.0)
- added TP11: TestPoint, TestPoint:TestPoint_Pad_D1.0mm, F.Cu at (111.4, 112.2)
- added TP110: FB, TestPoint:TestPoint_Pad_D1.0mm, F.Cu at (108.5, 46.0)
- added TP111: Vout, TestPoint:TestPoint_Pad_D1.0mm, F.Cu at (117.0, 36.5)
- added TP112: DVH1, TestPoint:TestPoint_Pad_D1.0mm, F.Cu at (103.5, 94.8)
- added TP113: DVL1, TestPoint:TestPoint_Pad_D1.0mm, F.Cu at (101.2, 94.8)
- added TP114: DVH2, TestPoint:TestPoint_Pad_D1.0mm, F.Cu at (101.8, 85.8)
- added TP115: DVL2, TestPoint:TestPoint_Pad_D1.0mm, F.Cu at (100.0, 85.8)
- added TP116: VH1, TestPoint:TestPoint_Pad_D1.0mm, F.Cu at (105.5, 99.8)
- added TP117: VL1, TestPoint:TestPoint_Pad_D1.0mm, F.Cu at (118.0, 99.5)
- added TP118: VH2, TestPoint:TestPoint_Pad_D1.0mm, F.Cu at (120.0, 85.5)
- added TP119: VL2, TestPoint:TestPoint_Pad_D1.0mm, F.Cu at (103.6, 85.7)
- added TP12: TestPoint, TestPoint:TestPoint_Pad_D1.0mm, F.Cu at (105.5, 112.2)
- added TP120: TestPoint, TestPoint:TestPoint_Pad_D1.0mm, F.Cu at (140.5, 104.8)
- added TP121: TestPoint, TestPoint:TestPoint_Pad_D1.0mm, F.Cu at (140.5, 96.0)
- added TP122: TH12, TestPoint:TestPoint_Pad_D1.0mm, F.Cu at (123.5, 111.0)
- added TP123: 1-2, TestPoint:TestPoint_Pad_D1.0mm, F.Cu at (133.0, 96.0)
- added TP124: TH1, TestPoint:TestPoint_Pad_D1.0mm, F.Cu at (129.2, 114.0)
- added TP125: TestPoint, TestPoint:TestPoint_Pad_D1.0mm, F.Cu at (157.8, 118.0)
- added TP126: TestPoint, TestPoint:TestPoint_Pad_D1.0mm, F.Cu at (156.2, 118.0)
- added TP127: TestPoint, TestPoint:TestPoint_Pad_D1.0mm, F.Cu at (157.8, 84.8)
- added TP128: TestPoint, TestPoint:TestPoint_Pad_D1.0mm, F.Cu at (156.2, 84.8)
- added TP129: TestPoint, TestPoint:TestPoint_Pad_D1.0mm, F.Cu at (148.0, 84.0)
- added TP13: TestPoint, TestPoint:TestPoint_Pad_D1.0mm, F.Cu at (105.5, 116.8)
- added TP130: TestPoint, TestPoint:TestPoint_Pad_D1.0mm, F.Cu at (143.5, 120.2)
- added TP131: TestPoint, TestPoint:TestPoint_Pad_D1.0mm, F.Cu at (154.0, 99.0)
- added TP132: TestPoint, TestPoint:TestPoint_Pad_D1.0mm, F.Cu at (176.2, 112.8)
- added TP133: TestPoint, TestPoint:TestPoint_Pad_D1.0mm, F.Cu at (166.5, 125.5)
- added TP134: TestPoint, TestPoint:TestPoint_Pad_D1.0mm, F.Cu at (173.8, 125.5)
- added TP135: TestPoint, TestPoint:TestPoint_Pad_D1.0mm, F.Cu at (176.2, 69.8)
- added TP136: TestPoint, TestPoint:TestPoint_Pad_D1.0mm, F.Cu at (166.5, 82.5)
- added TP137: TestPoint, TestPoint:TestPoint_Pad_D1.0mm, F.Cu at (173.8, 82.5)
- added TP138: TestPoint, TestPoint:TestPoint_Pad_D1.0mm, F.Cu at (176.2, 50.0)
- added TP139: TestPoint, TestPoint:TestPoint_Pad_D1.0mm, F.Cu at (166.5, 62.8)
- added TP14: TestPoint, TestPoint:TestPoint_Pad_D1.0mm, F.Cu at (109.6, 112.2)
- added TP140: TestPoint, TestPoint:TestPoint_Pad_D1.0mm, F.Cu at (173.8, 62.8)
- added TP141: DVH3, TestPoint:TestPoint_Pad_D1.0mm, F.Cu at (103.0, 71.0)
- added TP142: DVL3, TestPoint:TestPoint_Pad_D1.0mm, F.Cu at (101.2, 71.0)
- added TP143: DVH4, TestPoint:TestPoint_Pad_D1.0mm, F.Cu at (102.2, 62.0)
- added TP144: DVL4, TestPoint:TestPoint_Pad_D1.0mm, F.Cu at (100.5, 62.0)
- added TP145: VH3, TestPoint:TestPoint_Pad_D1.0mm, F.Cu at (104.0, 66.8)
- added TP146: VL3, TestPoint:TestPoint_Pad_D1.0mm, F.Cu at (118.2, 66.8)
- added TP147: VH4, TestPoint:TestPoint_Pad_D1.0mm, F.Cu at (118.0, 57.0)
- added TP148: VL4, TestPoint:TestPoint_Pad_D1.0mm, F.Cu at (105.5, 57.0)
- added TP149: TestPoint, TestPoint:TestPoint_Pad_D1.0mm, F.Cu at (140.5, 61.8)
- added TP15: TestPoint, TestPoint:TestPoint_Pad_D1.0mm, F.Cu at (110.5, 117.2)
- added TP150: TestPoint, TestPoint:TestPoint_Pad_D1.0mm, F.Cu at (140.5, 53.0)
- added TP151: TH34, TestPoint:TestPoint_Pad_D1.0mm, F.Cu at (123.5, 68.0)
- added TP152: 3-4, TestPoint:TestPoint_Pad_D1.0mm, F.Cu at (133.0, 53.0)
- added TP153: TH3, TestPoint:TestPoint_Pad_D1.0mm, F.Cu at (127.0, 72.5)
- added TP154: TestPoint, TestPoint:TestPoint_Pad_D1.0mm, F.Cu at (157.8, 75.0)
- added TP155: TestPoint, TestPoint:TestPoint_Pad_D1.0mm, F.Cu at (156.2, 75.0)
- added TP156: TestPoint, TestPoint:TestPoint_Pad_D1.0mm, F.Cu at (157.8, 41.8)
- added TP157: TestPoint, TestPoint:TestPoint_Pad_D1.0mm, F.Cu at (156.2, 41.8)
- added TP158: TestPoint, TestPoint:TestPoint_Pad_D1.0mm, F.Cu at (148.0, 41.0)
- added TP159: TestPoint, TestPoint:TestPoint_Pad_D1.0mm, F.Cu at (143.5, 77.2)
- added TP16: VIN, TestPoint:TestPoint_Pad_D1.0mm, F.Cu at (56.2, 59.8)
- added TP160: TestPoint, TestPoint:TestPoint_Pad_D1.0mm, F.Cu at (154.0, 56.0)
- added TP161: SS, TestPoint:TestPoint_Pad_D1.0mm, F.Cu at (68.8, 42.8)
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Routing:
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- added copper zone on F.Cu, net /+15V
- added copper zone on F.Cu, net /-15V
- added copper zone on F.Cu, net /3.3V
- added copper zone on F.Cu, net /Vin
- added copper zone on F.Cu, net /Vout
- added copper zone on F.Cu, net CHASSIS
- added copper zone on F.Cu, net GND
- added copper zone on In1.Cu, net GND
- added copper zone on In2.Cu, net GND
- added copper zone on F.Cu, net Net-(C43-Pad1)
- added copper zone on F.Cu, net Net-(C43-Pad2)
- added copper zone on F.Cu, net Net-(D30-Pad2)
- added copper zone on F.Cu, net Net-(D31-Pad1)
- added copper zone on F.Cu, net Net-(L2-Pad1)
Other:
- board outline added: 170 x 100 mm
- copper layers 2 -> 4
- net class Default: trace_width 0.25 -> 0.15; via_dia 0.8 -> 0.66; via_drill 0.4 -> 0.33
- net class Power added: clearance 0.2, trace_width 0.4, via_dia 0.812, via_drill 0.406
- rule pad_to_mask_clearance: 0.051 -> 0.08
- rule solder_mask_min_width: 0.25 -> 0.2
- rule trace_min: 0.2 -> 0.15
- rule via_min_drill: 0.3 -> 0.33
- rule via_min_size: 0.4 -> 0.635
- board text added: "02-13-2020"
- board text added: "BOOT"
- board text added: "DC IN 5-12V"
- board text added: "GND"
- board text added: "I/O 1 OC"
- board text added: "I/O 2 OC"
- board text added: "I/O 3 OC"
- board text added: "I/O 4 OC"
- board text added: "I/O MASTER v1.0"
- board text added: "IO1"
- board text added: "IO2"
- board text added: "IO3"
- board text added: "IO4"
- board text added: "RESET"
- board text added: "SWD/JTAG"
- board text added: "VOUT"
